File: STM32-Li-ion-charger-dischager-LCD.kicad_pcb (KiCad board)
At the start: 2 copper layers, 0 parts

Commit message: soft
Parts:
- added BT1: Battery_Cell, Connector_PinHeader_2.54mm:PinHeader_1x02_P2.54mm_Vertical, F.Cu at (139.7, 79.7)
- added BT2: Battery_Cell, Connector_PinHeader_2.54mm:PinHeader_1x02_P2.54mm_Vertical, F.Cu at (155.7, 64.9)
- added BT3: Battery_Cell, Connector_PinHeader_2.54mm:PinHeader_1x02_P2.54mm_Vertical, F.Cu at (142.7, 50.1)
- added C1: 10n, Capacitor_SMD:C_0603_1608Metric_Pad1.08x0.95mm_HandSolder, F.Cu at (96.4, 51.9)
- added C10: 24P, Capacitor_SMD:C_0603_1608Metric_Pad1.08x0.95mm_HandSolder, F.Cu at (107.0, 41.3)
- added C11: 24P, Capacitor_SMD:C_0603_1608Metric_Pad1.08x0.95mm_HandSolder, F.Cu at (107.0, 38.8)
- added C12: C_Small, Capacitor_SMD:C_0603_1608Metric_Pad1.08x0.95mm_HandSolder, F.Cu at (116.2, 36.8)
- added C13: 100n, Capacitor_SMD:C_0603_1608Metric_Pad1.08x0.95mm_HandSolder, F.Cu at (116.2, 34.3)
- added C14: 100n, Capacitor_SMD:C_0603_1608Metric_Pad1.08x0.95mm_HandSolder, F.Cu at (100.7, 51.9)
- added C15: 100n, Capacitor_SMD:C_0603_1608Metric_Pad1.08x0.95mm_HandSolder, F.Cu at (85.5, 59.2)
- added C16: 100n, Capacitor_SMD:C_0603_1608Metric_Pad1.08x0.95mm_HandSolder, F.Cu at (81.3, 61.8)
- added C18: 1u, Capacitor_SMD:C_0603_1608Metric_Pad1.08x0.95mm_HandSolder, F.Cu at (155.8, 78.6)
- added C19: 1u, Capacitor_SMD:C_0603_1608Metric_Pad1.08x0.95mm_HandSolder, F.Cu at (144.2, 83.6)
- added C2: 100n, Capacitor_SMD:C_0603_1608Metric_Pad1.08x0.95mm_HandSolder, F.Cu at (111.9, 34.3)
- added C21: 4.7u, Capacitor_SMD:C_0603_1608Metric_Pad1.08x0.95mm_HandSolder, F.Cu at (151.4, 76.5)
- added C22: 4.7u, Capacitor_SMD:C_0603_1608Metric_Pad1.08x0.95mm_HandSolder, F.Cu at (146.9, 86.6)
- added C23: 100n, Capacitor_SMD:C_0603_1608Metric_Pad1.08x0.95mm_HandSolder, F.Cu at (148.6, 81.5)
- added C24: 1u, Capacitor_SMD:C_0603_1608Metric_Pad1.08x0.95mm_HandSolder, F.Cu at (142.6, 56.2)
- added C25: 1u, Capacitor_SMD:C_0603_1608Metric_Pad1.08x0.95mm_HandSolder, F.Cu at (158.1, 46.3)
- added C26: 3.3, Capacitor_THT:CP_Radial_D8.0mm_P3.50mm, F.Cu at (149.4, 43.0)
- added C27: 3.3, Capacitor_THT:CP_Radial_D8.0mm_P3.50mm, F.Cu at (139.7, 43.0)
- added C3: 10n, Capacitor_SMD:C_0603_1608Metric_Pad1.08x0.95mm_HandSolder, F.Cu at (105.7, 43.8)
- added C4: 10n, Capacitor_SMD:C_0603_1608Metric_Pad1.08x0.95mm_HandSolder, F.Cu at (105.7, 46.3)
- added C5: 10n, Capacitor_SMD:C_0603_1608Metric_Pad1.08x0.95mm_HandSolder, F.Cu at (94.2, 59.2)
- added C6: 1u, Capacitor_SMD:C_0603_1608Metric_Pad1.08x0.95mm_HandSolder, F.Cu at (90.0, 61.7)
- added C7: 1u, Capacitor_SMD:C_0603_1608Metric_Pad1.08x0.95mm_HandSolder, F.Cu at (89.9, 59.2)
- added C8: 24P, Capacitor_SMD:C_0603_1608Metric_Pad1.08x0.95mm_HandSolder, F.Cu at (105.7, 48.8)
- added C9: 24P, Capacitor_SMD:C_0603_1608Metric_Pad1.08x0.95mm_HandSolder, F.Cu at (96.4, 54.4)
- added D1: LED_Small, LED_SMD:LED_0603_1608Metric_Pad1.05x0.95mm_HandSolder, F.Cu at (81.2, 56.8)
- added D2: LED_Small, LED_SMD:LED_0603_1608Metric_Pad1.05x0.95mm_HandSolder, F.Cu at (155.5, 71.1)
- added D3: LED_Small, LED_SMD:LED_0603_1608Metric_Pad1.05x0.95mm_HandSolder, F.Cu at (133.8, 85.8)
- added D4: LED_Small, LED_SMD:LED_0603_1608Metric_Pad1.05x0.95mm_HandSolder, F.Cu at (151.5, 74.0)
- added D5: LED_Small, LED_SMD:LED_0603_1608Metric_Pad1.05x0.95mm_HandSolder, F.Cu at (138.2, 85.8)
- added D6: D_Shockley, Diode_THT:D_A-405_P12.70mm_Horizontal, F.Cu at (126.0, 64.7)
- added D7: D_Shockley, Diode_THT:D_A-405_P12.70mm_Horizontal, F.Cu at (126.0, 35.2)
- added FB1: HI1806T600R-10, SamacSys_Parts:BEADC4516X185N, F.Cu at (75.6, 62.3)
- added FB2: HI1806T600R-10, SamacSys_Parts:BEADC4516X185N, F.Cu at (68.5, 62.3)
- added IC1: MCP73834T-FCI_UN, SamacSys_Parts:SOP50P490X110-10N, F.Cu at (128.0, 85.8)
- added IC2: MCP73834T-FCI_UN, SamacSys_Parts:SOP50P490X110-10N, F.Cu at (140.9, 75.0)
- added IC3: AP2112M-3.3TRG1, SamacSys_Parts:SOIC127P600X170-8N, F.Cu at (128.5, 80.2)
- added J1: Conn_01x10, Connector_PinHeader_2.54mm:PinHeader_1x10_P2.54mm_Vertical, F.Cu at (72.0, 35.4)
- added J10: Conn_01x02, Resistor_THT:R_Axial_DIN0309_L9.0mm_D3.2mm_P5.08mm_Vertical, F.Cu at (126.7, 55.4)
- added J2: Conn_01x10, Connector_PinHeader_2.54mm:PinHeader_1x10_P2.54mm_Vertical, F.Cu at (76.6, 35.4)
- added J3: Conn_01x10, Connector_PinHeader_2.54mm:PinHeader_1x10_P2.54mm_Vertical, F.Cu at (67.3, 35.4)
- added J4: Conn_01x08, Connector_PinHeader_2.54mm:PinHeader_1x08_P2.54mm_Vertical, F.Cu at (81.3, 35.4)
- added J6: Conn_01x02, Connector_PinHeader_2.54mm:PinHeader_1x02_P2.54mm_Vertical, F.Cu at (135.1, 79.7)
- added J7: Conn_01x02, Connector_PinHeader_2.54mm:PinHeader_1x02_P2.54mm_Vertical, F.Cu at (146.9, 75.0)
- added J8: Conn_01x03, Connector_PinHeader_2.54mm:PinHeader_1x03_P2.54mm_Vertical, F.Cu at (138.1, 50.1)
- added J9: Conn_01x02, Connector_Wago:Wago_734-132_1x02_P3.50mm_Vertical, F.Cu at (128.1, 47.6)
- added R1: 1k, Resistor_SMD:R_0603_1608Metric_Pad0.98x0.95mm_HandSolder, F.Cu at (85.6, 61.7)
- added R10: 470, Resistor_SMD:R_0603_1608Metric_Pad0.98x0.95mm_HandSolder, F.Cu at (152.9, 81.5)
- added R11: 10k, Resistor_SMD:R_0603_1608Metric_Pad0.98x0.95mm_HandSolder, F.Cu at (151.4, 79.0)
- added R12: 10k, Resistor_SMD:R_0603_1608Metric_Pad0.98x0.95mm_HandSolder, F.Cu at (142.6, 86.2)
- added R13: 47k, Resistor_SMD:R_0603_1608Metric_Pad0.98x0.95mm_HandSolder, F.Cu at (151.6, 53.5)
- added R14: 10k, Resistor_SMD:R_0603_1608Metric_Pad0.98x0.95mm_HandSolder, F.Cu at (156.7, 49.0)
- added R15: 10k, Resistor_SMD:R_0603_1608Metric_Pad0.98x0.95mm_HandSolder, F.Cu at (147.2, 53.5)
- added R16: 10k, Resistor_SMD:R_0603_1608Metric_Pad0.98x0.95mm_HandSolder, F.Cu at (146.9, 56.2)
- added R17: 5m, Resistor_SMD:R_0603_1608Metric_Pad0.98x0.95mm_HandSolder, F.Cu at (158.1, 43.8)
- added R18: 1m, Resistor_SMD:R_0603_1608Metric_Pad0.98x0.95mm_HandSolder, F.Cu at (152.3, 49.0)
- added R19: 50k, Resistor_SMD:R_0603_1608Metric_Pad0.98x0.95mm_HandSolder, F.Cu at (158.1, 41.3)
- added R2: 10k, Resistor_SMD:R_0603_1608Metric_Pad0.98x0.95mm_HandSolder, F.Cu at (111.3, 41.9)
- added R20: 5m, Resistor_SMD:R_0603_1608Metric_Pad0.98x0.95mm_HandSolder, F.Cu at (158.1, 38.8)
- added R22: 1M, Resistor_THT:R_Axial_DIN0411_L9.9mm_D3.6mm_P7.62mm_Vertical, F.Cu at (126.8, 39.9)
- added R23: 1M, Resistor_THT:R_Axial_DIN0411_L9.9mm_D3.6mm_P7.62mm_Vertical, F.Cu at (142.9, 35.6)
- added R3: 10k, Resistor_SMD:R_0603_1608Metric_Pad0.98x0.95mm_HandSolder, F.Cu at (81.1, 59.3)
- added R4: 10k, Resistor_SMD:R_0603_1608Metric_Pad0.98x0.95mm_HandSolder, F.Cu at (111.3, 39.3)
- added R5: 1k, Resistor_SMD:R_0603_1608Metric_Pad0.98x0.95mm_HandSolder, F.Cu at (111.9, 36.8)
- added R6: 10k, Resistor_SMD:R_0603_1608Metric_Pad0.98x0.95mm_HandSolder, F.Cu at (155.8, 73.6)
- added R7: 470, Resistor_SMD:R_0603_1608Metric_Pad0.98x0.95mm_HandSolder, F.Cu at (148.6, 84.1)
- added R8: 470, Resistor_SMD:R_0603_1608Metric_Pad0.98x0.95mm_HandSolder, F.Cu at (144.2, 81.1)
- added R9: 470, Resistor_SMD:R_0603_1608Metric_Pad0.98x0.95mm_HandSolder, F.Cu at (155.8, 76.1)
- added RV1: 4.7k, Z_mycustom_footprint_lib:2002102255, F.Cu at (141.3, 63.3)
- added RV2: 4.7k, Z_mycustom_footprint_lib:2002102255, F.Cu at (125.3, 67.6)
- added S1: PTS526_SK15_SMTR2_LFS, SamacSys_Parts:PTS526SK15SMTR2LFS, F.Cu at (89.2, 37.2)
- added S2: PTS526_SK15_SMTR2_LFS, SamacSys_Parts:PTS526SK15SMTR2LFS, F.Cu at (99.8, 37.2)
- added S3: PTS526_SK15_SMTR2_LFS, SamacSys_Parts:PTS526SK15SMTR2LFS, F.Cu at (89.2, 53.8)
- added S4: PTS526_SK15_SMTR2_LFS, SamacSys_Parts:PTS526SK15SMTR2LFS, F.Cu at (89.2, 45.5)
- added U1: STM32L151C6Ux, Package_DFN_QFN:QFN-48-1EP_7x7mm_P0.5mm_EP5.6x5.6mm, F.Cu at (98.9, 46.0)
- added U2: LM4040DBZ-3, Package_TO_SOT_SMD:SOT-23, F.Cu at (107.3, 35.3)
- added U3: OP179GRT, Package_TO_SOT_SMD:SOT-23-5, F.Cu at (147.6, 50.0)
- added U4: OP179GRT, Package_TO_SOT_SMD:SOT-23-5, F.Cu at (155.1, 35.3)
