File: STM32-Li-ion-charger-dischager-LCD.kicad_pcb (KiCad board)
At the start: 2 copper layers, 81 parts, among them IC1 MCP73834T-FCI_UN, IC2 MCP73834T-FCI_UN, IC3 AP2112M-3.3TRG1, J1 Conn_01x10, J10 Conn_01x02, J2 Conn_01x10, J3 Conn_01x10, J4 Conn_01x08, J6 Conn_01x02, J7 Conn_01x02, J8 Conn_01x03, J9 Conn_01x02, U1 STM32L151C6Ux, U2 LM4040DBZ-3, U3 OP179GRT, U4 OP179GRT

Commit message: t
Parts:
- removed J1, J2, J3: Conn_01x10, Connector_PinHeader_2.54mm:PinHeader_1x10_P2.54mm_Vertical
- added B1: ARDUINO_UNO_R3_SHIELDBASIC, Boards:UNO_R3_SHIELD, F.Cu at (196.7, 116.3)
- added C28: 100n, Capacitor_SMD:C_0603_1608Metric_Pad1.08x0.95mm_HandSolder, F.Cu at (63.0, 3.27)
- added C29: 1u, Capacitor_SMD:C_0603_1608Metric_Pad1.08x0.95mm_HandSolder, F.Cu at (110.2, 9.06)
- added C30: 100n, Capacitor_SMD:C_0603_1608Metric_Pad1.08x0.95mm_HandSolder, F.Cu at (16.6, 27.7)
- added C31: 100n, Capacitor_SMD:C_0603_1608Metric_Pad1.08x0.95mm_HandSolder, F.Cu at (7.88, 27.7)
- added C32: 100n, Capacitor_SMD:C_0603_1608Metric_Pad1.08x0.95mm_HandSolder, F.Cu at (24.7, 17.1)
- added C33: 100n, Capacitor_SMD:C_0603_1608Metric_Pad1.08x0.95mm_HandSolder, F.Cu at (24.7, 14.6)
- added J12: ARJM11C7-114-BA-EW2, SamacSys_Parts:ARJM11C7114BAEW2, F.Cu at (24.0, 115.9)
- added R24: 10k, Resistor_SMD:R_0603_1608Metric_Pad0.98x0.95mm_HandSolder, F.Cu at (3.53, 36.9)
- added R25: 50k, Resistor_SMD:R_0603_1608Metric_Pad0.98x0.95mm_HandSolder, F.Cu at (200.1, -64.4)
- added R26: 50k, Resistor_SMD:R_0603_1608Metric_Pad0.98x0.95mm_HandSolder, F.Cu at (188.7, -60.9)
- added R27: 50k, Resistor_SMD:R_0603_1608Metric_Pad0.98x0.95mm_HandSolder, F.Cu at (195.7, -64.4)
- added R28: 50k, Resistor_SMD:R_0603_1608Metric_Pad0.98x0.95mm_HandSolder, F.Cu at (193.0, -60.9)
- added R29: 330, Resistor_THT:R_Axial_DIN0411_L9.9mm_D3.6mm_P7.62mm_Vertical, F.Cu at (51.2, 4.59)
- added R30: 1k, Resistor_SMD:R_0603_1608Metric_Pad0.98x0.95mm_HandSolder, F.Cu at (55.2, 8.42)
- added R37: 50k, Resistor_SMD:R_0603_1608Metric_Pad0.98x0.95mm_HandSolder, F.Cu at (118.6, 2.61)
- added R38: 50k, Resistor_SMD:R_0603_1608Metric_Pad0.98x0.95mm_HandSolder, F.Cu at (123.2, -7.50)
- added R39: 50k, Resistor_SMD:R_0603_1608Metric_Pad0.98x0.95mm_HandSolder, F.Cu at (123.2, -4.99)
- added R40: 10k, Resistor_SMD:R_0603_1608Metric_Pad0.98x0.95mm_HandSolder, F.Cu at (110.2, -57.4)
- added R41: 10k, Resistor_SMD:R_0603_1608Metric_Pad0.98x0.95mm_HandSolder, F.Cu at (114.5, -59.9)
- added R42: 50k, Resistor_SMD:R_0603_1608Metric_Pad0.98x0.95mm_HandSolder, F.Cu at (119.4, -64.4)
- added R43: 50k, Resistor_SMD:R_0603_1608Metric_Pad0.98x0.95mm_HandSolder, F.Cu at (115.1, -64.4)
- added R45: 1k, Resistor_SMD:R_0603_1608Metric_Pad0.98x0.95mm_HandSolder, F.Cu at (110.2, -59.9)
- added R46: 50, Resistor_SMD:R_0603_1608Metric_Pad0.98x0.95mm_HandSolder, F.Cu at (12.2, 27.7)
- added R47: 330, Resistor_SMD:R_0603_1608Metric_Pad0.98x0.95mm_HandSolder, F.Cu at (36.1, 3.27)
- added R48: 330, Resistor_SMD:R_0603_1608Metric_Pad0.98x0.95mm_HandSolder, F.Cu at (3.53, 27.7)
- added R49: 50, Resistor_SMD:R_0603_1608Metric_Pad0.98x0.95mm_HandSolder, F.Cu at (36.1, 5.78)
- added R50: 50, Resistor_SMD:R_0603_1608Metric_Pad0.98x0.95mm_HandSolder, F.Cu at (24.7, 19.6)
- added R51: 50, Resistor_SMD:R_0603_1608Metric_Pad0.98x0.95mm_HandSolder, F.Cu at (40.4, 3.27)
- added R52: 10K, Resistor_SMD:R_0603_1608Metric_Pad0.98x0.95mm_HandSolder, F.Cu at (29.1, 14.6)
- added RV3: 47k, Z_mycustom_footprint_lib:2002102255, F.Cu at (109.0, -8.01)
- added U5: LM4040DBZ-3, Package_TO_SOT_SMD:SOT-23, F.Cu at (110.5, -63.4)
- added U6: W5500, Package_QFP:LQFP-48_7x7mm_P0.5mm, F.Cu at (28.2, 7.69)
- C1: value 10n -> 4u7
- C3, C4: value 10n -> 100n
- C7: value 1u -> 100n
- R1: value 1k -> 10k
- R17: value 5m -> 10k
- R18: value 1m -> 10k
- R20: value 5m -> 47k
- U2: value LM4040DBZ-3 -> OPA188xxD; footprint Package_TO_SOT_SMD:SOT-23 -> Package_SO:SOIC-8_3.9x4.9mm_P1.27mm
- moved FB1 170.4 mm to (190.0, -63.9)
- moved C6 153.6 mm to (188.7, -55.9)
- moved C5 150.9 mm to (188.7, -58.4)
- moved R1 86.6 mm to (3.53, 34.3)
- moved C7 64.1 mm to (50.8, 8.42)
- moved U2 31.1 mm to (112.2, 4.58)
Connections:
- net test_pwm renamed Net-(R13-Pad1)
- BT1 pad 1: ADC1 -> +BATT
- BT2 pad 1: ADC2 -> BATT2+
- BT3 pad 1: Net-(BT3-Pad1) -> /BattDischarger/Measured_BATT+
- C21 pad 1: ADC1 -> +BATT
- C22 pad 1: ADC2 -> BATT2+
- C7 pad 1: OpAmp_power -> Signal_out
- C7 pad 2: GND -> /BattDischarger/Measured_BATT+
- IC1 pad 10: ADC1 -> +BATT
- IC1 pad 9: ADC1 -> +BATT
- IC2 pad 10: ADC2 -> BATT2+
- IC2 pad 9: ADC2 -> BATT2+
- J8 pad 1: ADC1 -> BATT2+
- J8 pad 3: ADC2 -> +BATT
- J9 pad 2: Net-(BT3-Pad1) -> /BattDischarger/Measured_BATT+
- R1 pad 1: +3.3VA -> OpAmp_power
- R1 pad 2: ADC4 -> /NRST
- R17 pad 1: ADC3 -> ADC5
- R18 pad 1: Net-(JP2-Pad1) -> /BattDischarger/Measured_BATT+
- R18 pad 2: GND -> Net-(JP2-Pad1)
- R20 pad 1: Net-(BT3-Pad1) -> /BattDischarger/Measured_BATT+
- R20 pad 2: ADC3 -> ADC5
- U1 pad 24: unconnected-(U1-Pad24) -> OpAmp_power
- U1 pad 36: unconnected-(U1-Pad36) -> OpAmp_power
- U1 pad 44: unconnected-(U1-Pad44) -> /BOOT0
- U1 pad 48: unconnected-(U1-Pad48) -> OpAmp_power
- U1 pad 9: unconnected-(U1-Pad9) -> +3.3VA
- U2 pad 1: ADC4 -> unconnected-(U2-Pad1)
- U2 pad 2: GND -> ADC4
- U2 pad 3: (no net) -> Net-(R39-Pad1)
- U3 pad 3: Net-(C24-Pad1) -> Net-(U3-Pad3)
- U3 pad 4: ADC5 -> ADC6_load

Commit message: more work
Parts:
- added C34: 100n, Capacitor_SMD:C_0603_1608Metric_Pad1.08x0.95mm_HandSolder, F.Cu at (63.3, -17.6)
- added C35: 100n, Capacitor_SMD:C_0603_1608Metric_Pad1.08x0.95mm_HandSolder, F.Cu at (67.6, -17.2)
- added C36: 4.7u, Capacitor_SMD:C_0603_1608Metric_Pad1.08x0.95mm_HandSolder, F.Cu at (61.5, -10.1)
- added C37: 4.7u, Capacitor_SMD:C_0603_1608Metric_Pad1.08x0.95mm_HandSolder, F.Cu at (75.0, -27.8)
- added C38: 100n, Capacitor_SMD:C_0603_1608Metric_Pad1.08x0.95mm_HandSolder, F.Cu at (178.3, -45.0)
- added C39: 10u, Capacitor_SMD:C_0603_1608Metric_Pad1.08x0.95mm_HandSolder, F.Cu at (182.7, -45.0)
- added C40: 100n, Capacitor_SMD:C_0603_1608Metric_Pad1.08x0.95mm_HandSolder, F.Cu at (145.8, -25.6)
- added C41: 100n, Capacitor_SMD:C_0603_1608Metric_Pad1.08x0.95mm_HandSolder, F.Cu at (191.4, -50.1)
- added C42: 100n, Capacitor_SMD:C_0603_1608Metric_Pad1.08x0.95mm_HandSolder, F.Cu at (177.6, -41.3)
- added C43: 100n, Capacitor_SMD:C_0603_1608Metric_Pad1.08x0.95mm_HandSolder, F.Cu at (182.7, -52.6)
- added C44: 4u7, Capacitor_SMD:C_0603_1608Metric_Pad1.08x0.95mm_HandSolder, F.Cu at (178.3, -47.5)
- added C45: 100n, Capacitor_SMD:C_0603_1608Metric_Pad1.08x0.95mm_HandSolder, F.Cu at (181.9, -42.5)
- added C46: 100n, Capacitor_SMD:C_0603_1608Metric_Pad1.08x0.95mm_HandSolder, F.Cu at (150.2, -28.2)
- added C47: 100n, Capacitor_SMD:C_0603_1608Metric_Pad1.08x0.95mm_HandSolder, F.Cu at (158.9, -28.2)
- added C48: 100n, Capacitor_SMD:C_0603_1608Metric_Pad1.08x0.95mm_HandSolder, F.Cu at (181.9, -40.0)
- added C49: 10u, Capacitor_SMD:C_0603_1608Metric_Pad1.08x0.95mm_HandSolder, F.Cu at (178.3, -50.0)
- added C50: 1u, Capacitor_SMD:C_0603_1608Metric_Pad1.08x0.95mm_HandSolder, F.Cu at (228.2, -118.4)
- added C51: 1u, Capacitor_SMD:C_0603_1608Metric_Pad1.08x0.95mm_HandSolder, F.Cu at (236.8, -128.5)
- added C52: 1u, Capacitor_SMD:C_0603_1608Metric_Pad1.08x0.95mm_HandSolder, F.Cu at (223.8, -115.9)
- added D12: LED_Small, LED_SMD:LED_0603_1608Metric_Pad1.05x0.95mm_HandSolder, F.Cu at (201.5, -27.5)
- added D13: LED_Small, LED_SMD:LED_0603_1608Metric_Pad1.05x0.95mm_HandSolder, F.Cu at (178.4, -52.6)
- added D14: LED_Small, LED_SMD:LED_0603_1608Metric_Pad1.05x0.95mm_HandSolder, F.Cu at (145.8, -28.2)
- added D15: D_Shockley, Diode_THT:D_A-405_P12.70mm_Horizontal, F.Cu at (38.9, -36.7)
- added IC4: PEC12R-4230F-S0024, SamacSys_Parts:PEC12R4230FS0024, F.Cu at (148.9, -17.3)
- added J1: Conn_01x02, Connector_PinHeader_2.54mm:PinHeader_1x02_P2.54mm_Vertical, F.Cu at (213.1, -32.1)
- added J13: Conn_01x02, Connector_PinHeader_2.54mm:PinHeader_1x02_P2.54mm_Vertical, F.Cu at (68.6, -31.8)
- added R53: 10K, Resistor_SMD:R_0603_1608Metric_Pad0.98x0.95mm_HandSolder, F.Cu at (187.0, -45.1)
- added R54: 10K, Resistor_SMD:R_0603_1608Metric_Pad0.98x0.95mm_HandSolder, F.Cu at (167.0, -33.0)
- added R55: 10K, Resistor_SMD:R_0603_1608Metric_Pad0.98x0.95mm_HandSolder, F.Cu at (167.0, -30.4)
- added R57: 1k, Resistor_SMD:R_0603_1608Metric_Pad0.98x0.95mm_HandSolder, F.Cu at (187.1, -52.6)
- added R58: 1k, Resistor_SMD:R_0603_1608Metric_Pad0.98x0.95mm_HandSolder, F.Cu at (182.7, -50.0)
- added R59: 50k, Resistor_SMD:R_0603_1608Metric_Pad0.98x0.95mm_HandSolder, F.Cu at (202.4, -94.3)
- added R60: 50k, Resistor_SMD:R_0603_1608Metric_Pad0.98x0.95mm_HandSolder, F.Cu at (228.4, -124.6)
- added R61: 50k, Resistor_SMD:R_0603_1608Metric_Pad0.98x0.95mm_HandSolder, F.Cu at (241.2, -131.0)
- added R62: 50k, Resistor_SMD:R_0603_1608Metric_Pad0.98x0.95mm_HandSolder, F.Cu at (215.4, -105.5)
- added R63: 50k, Resistor_SMD:R_0603_1608Metric_Pad0.98x0.95mm_HandSolder, F.Cu at (232.7, -124.6)
- added R64: 50k, Resistor_SMD:R_0603_1608Metric_Pad0.98x0.95mm_HandSolder, F.Cu at (223.8, -118.4)
- added R65: 50k, Resistor_SMD:R_0603_1608Metric_Pad0.98x0.95mm_HandSolder, F.Cu at (210.8, -100.7)
- added R66: 50k, Resistor_SMD:R_0603_1608Metric_Pad0.98x0.95mm_HandSolder, F.Cu at (223.8, -120.9)
- added R67: 50k, Resistor_SMD:R_0603_1608Metric_Pad0.98x0.95mm_HandSolder, F.Cu at (236.8, -131.0)
- added R68: 10k, Resistor_SMD:R_0603_1608Metric_Pad0.98x0.95mm_HandSolder, F.Cu at (154.5, -128.5)
- added R69: 10k, Resistor_SMD:R_0603_1608Metric_Pad0.98x0.95mm_HandSolder, F.Cu at (150.7, -131.0)
- added R70: 10k, Resistor_SMD:R_0603_1608Metric_Pad0.98x0.95mm_HandSolder, F.Cu at (145.8, -119.1)
- added R71: 10k, Resistor_SMD:R_0603_1608Metric_Pad0.98x0.95mm_HandSolder, F.Cu at (150.1, -121.6)
- added R72: 10k, Resistor_SMD:R_0603_1608Metric_Pad0.98x0.95mm_HandSolder, F.Cu at (155.0, -131.0)
- added R73: 10k, Resistor_SMD:R_0603_1608Metric_Pad0.98x0.95mm_HandSolder, F.Cu at (145.8, -121.6)
- added RV4: 47k, Z_mycustom_footprint_lib:2002102255, F.Cu at (214.2, -131.6)
- added RV5: 47k, Z_mycustom_footprint_lib:2002102255, F.Cu at (201.2, -111.3)
- added RV6: 47k, Z_mycustom_footprint_lib:2002102255, F.Cu at (201.2, -131.6)
- added S5: PTS526_SK15_SMTR2_LFS, SamacSys_Parts:PTS526SK15SMTR2LFS, F.Cu at (170.4, -38.4)
- added U10: OPA188xxD, Package_SO:SOIC-8_3.9x4.9mm_P1.27mm, F.Cu at (217.4, -119.0)
- added U11: OPA188xxD, Package_SO:SOIC-8_3.9x4.9mm_P1.27mm, F.Cu at (204.4, -98.7)
- added U7: NE555P, Package_DIP:DIP-8_W7.62mm, F.Cu at (51.9, -26.6)
- added U8: OP179GRT, Package_TO_SOT_SMD:SOT-23-5, F.Cu at (223.1, -34.9)
- added U9: OPA188xxD, Package_SO:SOIC-8_3.9x4.9mm_P1.27mm, F.Cu at (230.4, -129.1)
- R17: value 10k -> 5k
- R18: value 10k -> 1k
- R19: value 50k -> 10K
- R20: value 47k -> 10k
- moved B1 254.5 mm to (64.6, -101.2)
- moved J12 215.1 mm to (159.9, -50.7)
- moved R48 198.3 mm to (187.0, -47.6)
- moved C7 196.9 mm to (239.4, -48.2)
- moved R46 186.3 mm to (182.7, -47.5)
- moved R29 175.8 mm to (217.9, -51.3)
- moved R30 170.8 mm to (221.9, -28.7)
- moved C30 165.3 mm to (171.3, -30.4)
- moved R50 163.6 mm to (177.6, -38.7)
- moved R49 161.0 mm to (187.0, -50.1)
- moved C28 157.9 mm to (217.6, -28.7)
- moved C29 157.4 mm to (215.4, -108.0)
- moved U2 157.4 mm to (217.4, -112.5)
- moved C31 156.9 mm to (154.5, -28.2)
- moved R37 156.6 mm to (223.8, -113.4)
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Connections:
- net /EthernetLAN/LED_G renamed /EthernetLAN+PoE/LED_G
- net /EthernetLAN/LED_Y renamed /EthernetLAN+PoE/LED_Y
- net /EthernetLAN/RXN renamed /EthernetLAN+PoE/RXN
- net /EthernetLAN/RXP renamed /EthernetLAN+PoE/RXP
- net /EthernetLAN/TXN renamed /EthernetLAN+PoE/TXN
- net /EthernetLAN/TXP renamed /EthernetLAN+PoE/TXP
- net /FanControl/Thermistor renamed thermistor
- net ADC5 renamed measured_batt_v
- net ADC6 renamed bat1_v
- net ADC6_load renamed measured_batt_I
- net ADC7 renamed bat2_v
- B1 pad 3.3V: unconnected-(B1-Pad3.3V) -> OpAmp_power
- B1 pad A0: unconnected-(B1-PadA0) -> LCD_CONTROL
- B1 pad A1: unconnected-(B1-PadA1) -> TOUCH_Y
- B1 pad A2: unconnected-(B1-PadA2) -> TOUCH_X
- B1 pad A3: unconnected-(B1-PadA3) -> LCD_CS
- B1 pad A4: unconnected-(B1-PadA4) -> LCD_RST
- B1 pad D10: unconnected-(B1-PadD10) -> /Display&SDcard/SPI_SS1
- B1 pad D11: unconnected-(B1-PadD11) -> SPI_MOSI
- B1 pad D12: unconnected-(B1-PadD12) -> SPI_MISO
- B1 pad D13: unconnected-(B1-PadD13) -> SPI_CLK
- B1 pad D2: unconnected-(B1-PadD2) -> LCD_D2
- B1 pad D3: unconnected-(B1-PadD3) -> LCD_D3
- B1 pad D4: unconnected-(B1-PadD4) -> LCD_D4
- B1 pad D5: unconnected-(B1-PadD5) -> LCD_D5
- B1 pad D6: unconnected-(B1-PadD6) -> LCD_D6
- B1 pad D7: unconnected-(B1-PadD7) -> LCD_D7
- B1 pad D8: unconnected-(B1-PadD8) -> LCD_D0
- B1 pad D9: unconnected-(B1-PadD9) -> LCD_D1
- B1 pad GND@: unconnected-(B1-PadGND@) -> GND
- J12 pad 1: unconnected-(J12-Pad1) -> /EthernetLAN+PoE/VC1-
- J12 pad 2: unconnected-(J12-Pad2) -> /EthernetLAN+PoE/VC2-
- J12 pad 6: unconnected-(J12-Pad6) -> /EthernetLAN+PoE/VC1+
- J12 pad 7: unconnected-(J12-Pad7) -> /EthernetLAN+PoE/VC2+
- J4 pad 5: UART_CTS -> unconnected-(J4-Pad5)
- J4 pad 6: UART_RTS -> unconnected-(J4-Pad6)
- R16 pad 1: Net-(R16-Pad1) -> OpAmp_power
- R16 pad 2: Net-(JP1-Pad2) -> /EthernetLAN+PoE/W5500_RST
- R18 pad 1: /BattDischarger/Measured_BATT+ -> Net-(JP2-Pad1)
- R18 pad 2: Net-(JP2-Pad1) -> GND
- R19 pad 1: Net-(Q2-Pad2) -> OpAmp_power
- R19 pad 2: Net-(R16-Pad1) -> Net-(R19-Pad2)
- U1 pad 10: unconnected-(U1-Pad10) -> ADC1
- U1 pad 11: unconnected-(U1-Pad11) -> ADC2
- U1 pad 12: unconnected-(U1-Pad12) -> ADC3
- U1 pad 13: unconnected-(U1-Pad13) -> ADC4
- U1 pad 14: unconnected-(U1-Pad14) -> DAC1
- U1 pad 15: unconnected-(U1-Pad15) -> DAC2
- U1 pad 26: unconnected-(U1-Pad26) -> SPI_CLK
- U1 pad 27: unconnected-(U1-Pad27) -> SPI_MISO
- U1 pad 28: unconnected-(U1-Pad28) -> SPI_MOSI
- U1 pad 39: unconnected-(U1-Pad39) -> SPI2_CLK
- U1 pad 40: unconnected-(U1-Pad40) -> SPI2_MISO
- U1 pad 41: unconnected-(U1-Pad41) -> SPI2_MOSI
- U1 pad 42: unconnected-(U1-Pad42) -> I2C_CLK
- U1 pad 43: unconnected-(U1-Pad43) -> I2C_SDA
- U2 pad 2: ADC4 -> scope1
- U2 pad 6: ADC4 -> scope1
- U3 pad 3: Net-(U3-Pad3) -> Net-(C24-Pad1)
- U4 pad 4: Net-(R16-Pad1) -> Net-(Q2-Pad2)
- U6 pad 10: unconnected-(U6-Pad10) -> Net-(R56-Pad1)
- U6 pad 11: Net-(U6-Pad11) -> +3.3VA
- U6 pad 15: Net-(U6-Pad11) -> +3.3VA
- U6 pad 17: Net-(U6-Pad11) -> +3.3VA
- U6 pad 20: unconnected-(U6-Pad20) -> Net-(C44-Pad1)
- U6 pad 21: Net-(U6-Pad11) -> +3.3VA
- U6 pad 22: unconnected-(U6-Pad22) -> Net-(C43-Pad1)
- U6 pad 24: unconnected-(U6-Pad24) -> /EthernetLAN+PoE/spd_led
- U6 pad 26: unconnected-(U6-Pad26) -> /EthernetLAN+PoE/dup_led
- U6 pad 28: unconnected-(U6-Pad28) -> OpAmp_power
- U6 pad 30: unconnected-(U6-Pad30) -> Net-(U6-Pad30)
- U6 pad 31: unconnected-(U6-Pad31) -> Net-(U6-Pad31)
- U6 pad 32: unconnected-(U6-Pad32) -> /EthernetLAN+PoE/SPI2_SS
- U6 pad 33: unconnected-(U6-Pad33) -> SPI2_MOSI
- U6 pad 34: unconnected-(U6-Pad34) -> SPI2_MISO
- U6 pad 35: unconnected-(U6-Pad35) -> SPI2_CLK
- U6 pad 36: unconnected-(U6-Pad36) -> Net-(R55-Pad2)
- U6 pad 37: unconnected-(U6-Pad37) -> /EthernetLAN+PoE/W5500_RST
- U6 pad 4: Net-(U6-Pad11) -> +3.3VA
- U6 pad 43: unconnected-(U6-Pad43) -> Net-(R19-Pad2)
- U6 pad 44: unconnected-(U6-Pad44) -> Net-(R53-Pad2)
- U6 pad 45: unconnected-(U6-Pad45) -> Net-(R54-Pad2)
- U6 pad 8: Net-(U6-Pad11) -> +3.3VA

Commit message: h
Parts:
- removed B1: ARDUINO_UNO_R3_SHIELDBASIC, Boards:UNO_R3_SHIELD
- removed BT1, BT2, BT3: Battery_Cell, Connector_PinHeader_2.54mm:PinHeader_1x02_P2.54mm_Vertical
- removed C1, C44: 4u7, Capacitor_SMD:C_0603_1608Metric_Pad1.08x0.95mm_HandSolder
- removed C10, C11, C8, C9: 24P, Capacitor_SMD:C_0603_1608Metric_Pad1.08x0.95mm_HandSolder
- removed C12: C_Small, Capacitor_SMD:C_0603_1608Metric_Pad1.08x0.95mm_HandSolder
- removed C13, C14, C15, C16, C2, C23, C28, C3, C30, C31, C32, C33, C34, C35, C38, C4, C40, C41, C42, C43, C45, C46, C47, C48, C7: 100n, Capacitor_SMD:C_0603_1608Metric_Pad1.08x0.95mm_HandSolder
- removed C18, C19, C24, C25, C29, C50, C51, C52, C6: 1u, Capacitor_SMD:C_0603_1608Metric_Pad1.08x0.95mm_HandSolder
- removed C21, C22, C36, C37: 4.7u, Capacitor_SMD:C_0603_1608Metric_Pad1.08x0.95mm_HandSolder
- removed C26, C27: 3.3, Capacitor_THT:CP_Radial_D8.0mm_P3.50mm
- removed C39, C49: 10u, Capacitor_SMD:C_0603_1608Metric_Pad1.08x0.95mm_HandSolder
- removed C5: 10n, Capacitor_SMD:C_0603_1608Metric_Pad1.08x0.95mm_HandSolder
- removed D1, D12, D13, D14, D2, D3, D4, D5: LED_Small, LED_SMD:LED_0603_1608Metric_Pad1.05x0.95mm_HandSolder
- removed D15, D6, D7: D_Shockley, Diode_THT:D_A-405_P12.70mm_Horizontal
- removed FB1, FB2: HI1806T600R-10, SamacSys_Parts:BEADC4516X185N
- removed IC1, IC2: MCP73834T-FCI_UN, SamacSys_Parts:SOP50P490X110-10N
- removed IC3: AP2112M-3.3TRG1, SamacSys_Parts:SOIC127P600X170-8N
- removed IC4: PEC12R-4230F-S0024, SamacSys_Parts:PEC12R4230FS0024
- removed J1, J13, J6, J7: Conn_01x02, Connector_PinHeader_2.54mm:PinHeader_1x02_P2.54mm_Vertical
- removed J10: Conn_01x02, Resistor_THT:R_Axial_DIN0309_L9.0mm_D3.2mm_P5.08mm_Vertical
- removed J12: ARJM11C7-114-BA-EW2, SamacSys_Parts:ARJM11C7114BAEW2
- removed J4: Conn_01x08, Connector_PinHeader_2.54mm:PinHeader_1x08_P2.54mm_Vertical
- removed J8: Conn_01x03, Connector_PinHeader_2.54mm:PinHeader_1x03_P2.54mm_Vertical
- removed J9: Conn_01x02, Connector_Wago:Wago_734-132_1x02_P3.50mm_Vertical
- removed R1, R11, R12, R14, R15, R16, R2, R20, R24, R3, R4, R40, R41, R6, R68, R69, R70, R71, R72, R73: 10k, Resistor_SMD:R_0603_1608Metric_Pad0.98x0.95mm_HandSolder
- removed R10, R7, R8, R9: 470, Resistor_SMD:R_0603_1608Metric_Pad0.98x0.95mm_HandSolder
- removed R13: 47k, Resistor_SMD:R_0603_1608Metric_Pad0.98x0.95mm_HandSolder
- removed R17: 5k, Resistor_SMD:R_0603_1608Metric_Pad0.98x0.95mm_HandSolder
- removed R18, R30, R45, R5, R57, R58: 1k, Resistor_SMD:R_0603_1608Metric_Pad0.98x0.95mm_HandSolder
- removed R19, R52, R53, R54, R55: 10K, Resistor_SMD:R_0603_1608Metric_Pad0.98x0.95mm_HandSolder
- removed R22, R23: 1M, Resistor_THT:R_Axial_DIN0411_L9.9mm_D3.6mm_P7.62mm_Vertical
- removed R25, R26, R27, R28, R37, R38, R39, R42, R43, R59, R60, R61, R62, R63, R64, R65, R66, R67: 50k, Resistor_SMD:R_0603_1608Metric_Pad0.98x0.95mm_HandSolder
- removed R29: 330, Resistor_THT:R_Axial_DIN0411_L9.9mm_D3.6mm_P7.62mm_Vertical
- removed R46, R49, R50, R51: 50, Resistor_SMD:R_0603_1608Metric_Pad0.98x0.95mm_HandSolder
- removed R47, R48: 330, Resistor_SMD:R_0603_1608Metric_Pad0.98x0.95mm_HandSolder
- removed RV1, RV2: 4.7k, Z_mycustom_footprint_lib:2002102255
- removed RV3, RV4, RV5, RV6: 47k, Z_mycustom_footprint_lib:2002102255
- removed S1, S2, S3, S4, S5: PTS526_SK15_SMTR2_LFS, SamacSys_Parts:PTS526SK15SMTR2LFS
- removed U1: STM32L151C6Ux, Package_DFN_QFN:QFN-48-1EP_7x7mm_P0.5mm_EP5.6x5.6mm
- removed U10, U11, U2, U9: OPA188xxD, Package_SO:SOIC-8_3.9x4.9mm_P1.27mm
- removed U3, U4, U8: OP179GRT, Package_TO_SOT_SMD:SOT-23-5
- removed U5: LM4040DBZ-3, Package_TO_SOT_SMD:SOT-23
- removed U6: W5500, Package_QFP:LQFP-48_7x7mm_P0.5mm
- removed U7: NE555P, Package_DIP:DIP-8_W7.62mm
- added B501: ARDUINO_UNO_R3_SHIELDBASIC, Boards:UNO_R3_SHIELD, F.Cu at (178.1, -44.7)
- added BT201: Battery_Cell, Connector_PinHeader_2.54mm:PinHeader_1x02_P2.54mm_Vertical, F.Cu at (179.7, 54.9)
- added BT301: Battery_Cell, Connector_PinHeader_2.54mm:PinHeader_1x02_P2.54mm_Vertical, F.Cu at (270.9, -73.5)
- added BT901: Battery_Cell, Z_mycustom_footprint_lib:BATHLD001THM, F.Cu at (352.9, -66.1)
- added C101: 24P, Capacitor_SMD:C_0603_1608Metric_Pad1.08x0.95mm_HandSolder, F.Cu at (441.6, -51.9)
- added C102: 24P, Capacitor_SMD:C_0603_1608Metric_Pad1.08x0.95mm_HandSolder, F.Cu at (455.2, -63.6)
- added C103: 4u7, Capacitor_SMD:C_0603_1608Metric_Pad1.08x0.95mm_HandSolder, F.Cu at (455.2, -66.1)
- added C104: 24P, Capacitor_SMD:C_0603_1608Metric_Pad1.08x0.95mm_HandSolder, F.Cu at (450.9, -61.1)
- added C105: 24P, Capacitor_SMD:C_0603_1608Metric_Pad1.08x0.95mm_HandSolder, F.Cu at (452.2, -71.1)
- added C106: 100n, Capacitor_SMD:C_0603_1608Metric_Pad1.08x0.95mm_HandSolder, F.Cu at (463.6, -74.6)
- added C107: 100n, Capacitor_SMD:C_0603_1608Metric_Pad1.08x0.95mm_HandSolder, F.Cu at (460.9, -69.5)
- added C108: 100n, Capacitor_SMD:C_0603_1608Metric_Pad1.08x0.95mm_HandSolder, F.Cu at (441.6, -57.0)
- added C109: 100n, Capacitor_SMD:C_0603_1608Metric_Pad1.08x0.95mm_HandSolder, F.Cu at (459.2, -74.6)
- added C110: C_Small, Capacitor_SMD:C_0603_1608Metric_Pad1.08x0.95mm_HandSolder, F.Cu at (456.5, -71.1)
- added C111: 100n, Capacitor_SMD:C_0603_1608Metric_Pad1.08x0.95mm_HandSolder, F.Cu at (445.9, -54.5)
- added C112: 100n, Capacitor_SMD:C_0603_1608Metric_Pad1.08x0.95mm_HandSolder, F.Cu at (450.9, -66.1)
- added C113: 100n, Capacitor_SMD:C_0603_1608Metric_Pad1.08x0.95mm_HandSolder, F.Cu at (445.9, -57.0)
- added C201: 4.7u, Capacitor_SMD:C_0603_1608Metric_Pad1.08x0.95mm_HandSolder, F.Cu at (206.7, 54.3)
- added C202: 4.7u, Capacitor_SMD:C_0603_1608Metric_Pad1.08x0.95mm_HandSolder, F.Cu at (205.7, 61.8)
- added C203: 1u, Capacitor_SMD:C_0805_2012Metric_Pad1.18x1.45mm_HandSolder, F.Cu at (223.2, 43.4)
- added C204: 1u, Capacitor_SMD:C_0805_2012Metric_Pad1.18x1.45mm_HandSolder, F.Cu at (223.2, 46.4)
- added C205: 10n, Capacitor_SMD:C_0603_1608Metric_Pad1.08x0.95mm_HandSolder, F.Cu at (206.6, 56.8)
- added C206: 1u, Capacitor_SMD:C_0603_1608Metric_Pad1.08x0.95mm_HandSolder, F.Cu at (202.2, 57.9)
- added C207: 100n, Capacitor_SMD:C_0603_1608Metric_Pad1.08x0.95mm_HandSolder, F.Cu at (206.7, 51.8)
- added C208: 100n, Capacitor_SMD:C_0603_1608Metric_Pad1.08x0.95mm_HandSolder, F.Cu at (179.6, 61.8)
- added C209: 4.7u, Capacitor_SMD:C_0603_1608Metric_Pad1.08x0.95mm_HandSolder, F.Cu at (197.0, 60.4)
- added C210: 4.7u, Capacitor_SMD:C_0603_1608Metric_Pad1.08x0.95mm_HandSolder, F.Cu at (211.0, 52.9)
- added C301: 1u, Capacitor_SMD:C_0603_1608Metric_Pad1.08x0.95mm_HandSolder, F.Cu at (263.9, -64.0)
- added C302: 1u, Capacitor_SMD:C_0603_1608Metric_Pad1.08x0.95mm_HandSolder, F.Cu at (280.0, -74.6)
- added C303: 100n, Capacitor_SMD:C_0603_1608Metric_Pad1.08x0.95mm_HandSolder, F.Cu at (268.3, -64.0)
- added C304: 100n, Capacitor_SMD:C_0603_1608Metric_Pad1.08x0.95mm_HandSolder, F.Cu at (263.9, -61.5)
- added C401: 1u, Capacitor_SMD:C_0603_1608Metric_Pad1.08x0.95mm_HandSolder, F.Cu at (273.3, 40.2)
- added C402: 1u, Capacitor_SMD:C_0603_1608Metric_Pad1.08x0.95mm_HandSolder, F.Cu at (269.0, 45.2)
- added C403: 1u, Capacitor_SMD:C_0603_1608Metric_Pad1.08x0.95mm_HandSolder, F.Cu at (269.0, 42.7)
- added C404: 1u, Capacitor_SMD:C_0603_1608Metric_Pad1.08x0.95mm_HandSolder, F.Cu at (282.0, 30.0)
- added C801: 22u, Capacitor_THT:CP_Radial_D5.0mm_P2.00mm, F.Cu at (343.0, 12.2)
- added C802: 22p optional, Capacitor_SMD:C_0603_1608Metric_Pad1.08x0.95mm_HandSolder, F.Cu at (348.9, 17.0)
- added C803: 22u, Capacitor_THT:CP_Radial_D5.0mm_P2.00mm, F.Cu at (351.0, 5.90)
- added C804: 22u, Capacitor_THT:CP_Radial_D5.0mm_P2.00mm, F.Cu at (349.6, 12.5)
- added C901: 15pF, Capacitor_SMD:C_0603_1608Metric_Pad1.08x0.95mm_HandSolder, F.Cu at (342.8, -50.1)
- added C902: 15pF, Capacitor_SMD:C_0603_1608Metric_Pad1.08x0.95mm_HandSolder, F.Cu at (351.6, -54.7)
- added D101: LED_Small, LED_SMD:LED_0603_1608Metric_Pad1.05x0.95mm_HandSolder, F.Cu at (426.4, -52.1)
- added D201: LED_Small, LED_SMD:LED_0603_1608Metric_Pad1.05x0.95mm_HandSolder, F.Cu at (202.3, 46.6)
- added D202: LED_Small, LED_SMD:LED_0603_1608Metric_Pad1.05x0.95mm_HandSolder, F.Cu at (198.0, 50.4)
- added D203: LED_Small, LED_SMD:LED_0603_1608Metric_Pad1.05x0.95mm_HandSolder, F.Cu at (206.7, 49.2)
- added D204: LED_Small, LED_SMD:LED_0603_1608Metric_Pad1.05x0.95mm_HandSolder, F.Cu at (206.7, 46.6)
- added D205: D_Shockley, Diode_THT:D_DO-15_P15.24mm_Horizontal, F.Cu at (152.7, 44.4)
- added D206: D_Shockley, Diode_THT:D_A-405_P12.70mm_Horizontal, F.Cu at (171.6, 44.0)
- added D207: LED_Small Green, LED_SMD:LED_0603_1608Metric_Pad1.05x0.95mm_HandSolder, F.Cu at (193.6, 52.1)
- added D208: LED_Small Green, LED_SMD:LED_0603_1608Metric_Pad1.05x0.95mm_HandSolder, F.Cu at (202.3, 49.2)
- added D211: LED_Small Green, LED_SMD:LED_0603_1608Metric_Pad1.05x0.95mm_HandSolder, F.Cu at (211.1, 47.8)
- added D302: LED_Small, LED_SMD:LED_0603_1608Metric_Pad1.05x0.95mm_HandSolder, F.Cu at (259.3, -54.3)
- added F201: Polyfuse_Small, Fuse:Fuse_1812_4532Metric_Pad1.30x3.40mm_HandSolder, F.Cu at (169.1, 67.6)
- added FB101: HI1806T600R-10, SamacSys_Parts:BEADC4516X185N, F.Cu at (453.5, -74.1)
- added FB201: HI1806T600R-10, SamacSys_Parts:BEADC4516X185N, F.Cu at (199.5, 43.6)
- added FB202: HI1806T600R-10, SamacSys_Parts:BEADC4516X185N, F.Cu at (206.6, 43.6)
- added IC201: MCP73834T-FCI_UN, SamacSys_Parts:SOP50P490X110-10N, F.Cu at (161.8, 71.2)
- added IC202: MCP73834T-FCI_UN, SamacSys_Parts:SOP50P490X110-10N, F.Cu at (154.4, 71.2)
- added IC203: ISL9120IIAZ-TR5696, SamacSys_Parts:BGA9C40P3X3_141X141X55, F.Cu at (218.2, 48.6)
- added IC204: AP2112M-3.3TRG1, SamacSys_Parts:SOIC127P600X170-8N, F.Cu at (180.9, 49.4)
- added IC701: XRA1203IG24TR-F, SamacSys_Parts:SOP65P640X120-24N, F.Cu at (182.9, 81.7)
- added IC702: PEC12R-4230F-S0024, SamacSys_Parts:PEC12R4230FS0024, F.Cu at (157.9, 80.9)
- added J101: Conn_01x08, Connector_PinHeader_2.54mm:PinHeader_1x08_P2.54mm_Vertical, F.Cu at (426.5, -73.5)
- added J201: Conn_01x02_Male, Connector_PinHeader_2.54mm:PinHeader_1x02_P2.54mm_Vertical, F.Cu at (175.1, 60.9)
- added J202: Conn_01x02, Connector_PinHeader_2.54mm:PinHeader_1x02_P2.54mm_Vertical, F.Cu at (184.4, 54.9)
- added J203: Conn_01x02, Connector_PinHeader_2.54mm:PinHeader_1x02_P2.54mm_Vertical, F.Cu at (189.0, 53.9)
- added J204: Conn_01x02, Connector_PinHeader_2.54mm:PinHeader_1x02_P2.54mm_Vertical, F.Cu at (193.7, 44.2)
- added J205: USB_B_Mini, Connector_USB:USB_Mini-B_Lumberg_2486_01_Horizontal, F.Cu at (170.2, 51.7)
- added J206: Conn_01x03, Connector_PinHeader_2.54mm:PinHeader_1x03_P2.54mm_Vertical, F.Cu at (188.3, 44.2)
- added J301: Conn_01x02, Connector_PinHeader_2.54mm:PinHeader_1x02_P2.54mm_Vertical, F.Cu at (275.5, -73.5)
- added J302: Conn_01x03, Connector_PinHeader_2.54mm:PinHeader_1x03_P2.54mm_Vertical, F.Cu at (259.4, -62.9)
- added J303: Conn_01x02, Connector_Wago:Wago_734-132_1x02_P3.50mm_Vertical, F.Cu at (260.9, -70.6)
- added JP701: J1, Jumper:SolderJumper-2_P1.3mm_Open_RoundedPad1.0x1.5mm, F.Cu at (193.9, 78.8)
- added JP702: J1, Jumper:SolderJumper-2_P1.3mm_Open_RoundedPad1.0x1.5mm, F.Cu at (189.6, 83.8)
- added L801: NRH3012T2R2MN 2,2uH, SamacSys_Parts:NRH3012T220MNV, F.Cu at (343.7, 18.5)
- added Q201: DMG9933USD-13, SamacSys_Parts:SOIC127P600X175-8N, F.Cu at (165.8, 61.9)
- added R101: 10k, Resistor_SMD:R_0603_1608Metric_Pad0.98x0.95mm_HandSolder, F.Cu at (450.9, -63.6)
- added R102: 10k, Resistor_SMD:R_0603_1608Metric_Pad0.98x0.95mm_HandSolder, F.Cu at (445.9, -51.9)
- added R103: 10k, Resistor_SMD:R_0603_1608Metric_Pad0.98x0.95mm_HandSolder, F.Cu at (455.2, -61.1)
- added R104: 10k, Resistor_SMD:R_0603_1608Metric_Pad0.98x0.95mm_HandSolder, F.Cu at (441.6, -54.5)
- added R105: 10k, Resistor_SMD:R_0603_1608Metric_Pad0.98x0.95mm_HandSolder, F.Cu at (460.9, -67.0)
- added R106: 1k, Resistor_SMD:R_0603_1608Metric_Pad0.98x0.95mm_HandSolder, F.Cu at (452.2, -68.6)
- added R107: 10k, Resistor_SMD:R_0603_1608Metric_Pad0.98x0.95mm_HandSolder, F.Cu at (467.9, -74.6)
- added R108: 10k, Resistor_SMD:R_0603_1608Metric_Pad0.98x0.95mm_HandSolder, F.Cu at (460.9, -72.0)
- added R109: 10k, Resistor_SMD:R_0603_1608Metric_Pad0.98x0.95mm_HandSolder, F.Cu at (456.5, -68.6)
- added R110: 10k, Resistor_SMD:R_0603_1608Metric_Pad0.98x0.95mm_HandSolder, F.Cu at (465.2, -72.0)
- added R111: 10k, Resistor_SMD:R_0603_1608Metric_Pad0.98x0.95mm_HandSolder, F.Cu at (450.3, -57.0)
- added R201: 470, Resistor_SMD:R_0603_1608Metric_Pad0.98x0.95mm_HandSolder, F.Cu at (211.0, 55.4)
- added R202: 470, Resistor_SMD:R_0603_1608Metric_Pad0.98x0.95mm_HandSolder, F.Cu at (210.9, 57.9)
- added R203: 470, Resistor_SMD:R_0603_1608Metric_Pad0.98x0.95mm_HandSolder, F.Cu at (215.4, 52.9)
- added R204: 470, Resistor_SMD:R_0603_1608Metric_Pad0.98x0.95mm_HandSolder, F.Cu at (183.9, 61.1)
- added R205: 10k, Resistor_SMD:R_0603_1608Metric_Pad0.98x0.95mm_HandSolder, F.Cu at (197.9, 54.7)
- added R206: 10k, Resistor_SMD:R_0603_1608Metric_Pad0.98x0.95mm_HandSolder, F.Cu at (206.6, 59.3)
- added R207: 10k, Resistor_SMD:R_0603_1608Metric_Pad0.98x0.95mm_HandSolder, F.Cu at (192.6, 60.4)
- added R208: 10k, Resistor_SMD:R_0603_1608Metric_Pad0.98x0.95mm_HandSolder, F.Cu at (188.3, 61.1)
- added R209: 50k, Resistor_SMD:R_0603_1608Metric_Pad0.98x0.95mm_HandSolder, F.Cu at (197.0, 62.9)
- added R210: 50k, Resistor_SMD:R_0603_1608Metric_Pad0.98x0.95mm_HandSolder, F.Cu at (201.3, 62.9)
- added R211: 50k, Resistor_SMD:R_0603_1608Metric_Pad0.98x0.95mm_HandSolder, F.Cu at (211.1, 50.4)
- added R212: 50k, Resistor_SMD:R_0603_1608Metric_Pad0.98x0.95mm_HandSolder, F.Cu at (193.5, 57.9)
- added R213: 10k+ pullup, Resistor_SMD:R_0603_1608Metric_Pad0.98x0.95mm_HandSolder, F.Cu at (202.3, 52.9)
- added R214: 10k, Resistor_SMD:R_0603_1608Metric_Pad0.98x0.95mm_HandSolder, F.Cu at (197.9, 57.2)
- added R215: 10k, Resistor_SMD:R_0603_1608Metric_Pad0.98x0.95mm_HandSolder, F.Cu at (192.6, 62.9)
- added R216: 330, Resistor_SMD:R_0603_1608Metric_Pad0.98x0.95mm_HandSolder, F.Cu at (201.3, 60.4)
- added R217: 330, Resistor_SMD:R_0603_1608Metric_Pad0.98x0.95mm_HandSolder, F.Cu at (202.2, 55.4)
- added R301: 47k, Resistor_SMD:R_0603_1608Metric_Pad0.98x0.95mm_HandSolder, F.Cu at (263.9, -56.5)
- added R302: 10k, Resistor_SMD:R_0603_1608Metric_Pad0.98x0.95mm_HandSolder, F.Cu at (280.0, -72.0)
- added R303: 10k, Resistor_SMD:R_0603_1608Metric_Pad0.98x0.95mm_HandSolder, F.Cu at (275.1, -67.4)
- added R304: 5k, Resistor_SMD:R_0603_1608Metric_Pad0.98x0.95mm_HandSolder, F.Cu at (263.9, -59.0)
- added R305: 1k, Resistor_SMD:R_0603_1608Metric_Pad0.98x0.95mm_HandSolder, F.Cu at (268.3, -61.5)
- added R306: 10k, Resistor_SMD:R_0603_1608Metric_Pad0.98x0.95mm_HandSolder, F.Cu at (270.7, -67.4)
- added R308: 1k, Resistor_SMD:R_0603_1608Metric_Pad0.98x0.95mm_HandSolder, F.Cu at (268.3, -59.0)
- added R401: 50k, Resistor_SMD:R_0603_1608Metric_Pad0.98x0.95mm_HandSolder, F.Cu at (282.0, 32.6)
- added R402: 50k, Resistor_SMD:R_0603_1608Metric_Pad0.98x0.95mm_HandSolder, F.Cu at (256.0, 60.4)
- added R403: 50k, Resistor_SMD:R_0603_1608Metric_Pad0.98x0.95mm_HandSolder, F.Cu at (269.0, 47.7)
- added R404: 50k, Resistor_SMD:R_0603_1608Metric_Pad0.98x0.95mm_HandSolder, F.Cu at (269.0, 40.2)
- added R601: 10k, Resistor_SMD:R_0603_1608Metric_Pad0.98x0.95mm_HandSolder, F.Cu at (259.3, -41.4)
- added R602: 10k, Resistor_SMD:R_0603_1608Metric_Pad0.98x0.95mm_HandSolder, F.Cu at (263.6, -43.9)
- added R603: 50k, Resistor_SMD:R_0603_1608Metric_Pad0.98x0.95mm_HandSolder, F.Cu at (268.5, -48.4)
- added R604: 50k, Resistor_SMD:R_0603_1608Metric_Pad0.98x0.95mm_HandSolder, F.Cu at (264.2, -48.4)
- added R606: 1k, Resistor_SMD:R_0603_1608Metric_Pad0.98x0.95mm_HandSolder, F.Cu at (259.3, -43.9)
- added R701: 10k, Resistor_SMD:R_0603_1608Metric_Pad0.98x0.95mm_HandSolder, F.Cu at (180.6, 87.7)
- added R702: 10k, Resistor_SMD:R_0603_1608Metric_Pad0.98x0.95mm_HandSolder, F.Cu at (189.6, 78.2)
- added R703: 10k, Resistor_SMD:R_0603_1608Metric_Pad0.98x0.95mm_HandSolder, F.Cu at (185.0, 87.7)
- added R704: 10k, Resistor_SMD:R_0603_1608Metric_Pad0.98x0.95mm_HandSolder, F.Cu at (180.6, 90.2)
- added R705: 10k, Resistor_SMD:R_0603_1608Metric_Pad0.98x0.95mm_HandSolder, F.Cu at (189.6, 80.8)
- added RR801: R_Small, Resistor_THT:R_Axial_DIN0204_L3.6mm_D1.6mm_P5.08mm_Horizontal, F.Cu at (342.1, 7.35)
- added RR802: R_Small, Resistor_THT:R_Axial_DIN0204_L3.6mm_D1.6mm_P5.08mm_Horizontal, F.Cu at (342.1, 4.20)
- added RV201: 10k, Z_mycustom_footprint_lib:2002102255, F.Cu at (233.3, 36.7)
- added RV202: 10k, Z_mycustom_footprint_lib:2002102255, F.Cu at (151.8, 47.8)
- added RV401: 47k, Z_mycustom_footprint_lib:2002102255, F.Cu at (267.8, 29.5)
- added RV402: 47k, Z_mycustom_footprint_lib:2002102255, F.Cu at (254.8, 49.8)
- added RV403: 47k, Z_mycustom_footprint_lib:2002102255, F.Cu at (254.8, 39.6)
- added RV404: 47k, Z_mycustom_footprint_lib:2002102255, F.Cu at (254.8, 29.5)
- added S101: PTS526_SK15_SMTR2_LFS, SamacSys_Parts:PTS526SK15SMTR2LFS, F.Cu at (434.3, -71.7)
- added S102: PTS526_SK15_SMTR2_LFS, SamacSys_Parts:PTS526SK15SMTR2LFS, F.Cu at (434.3, -55.1)
- added S103: PTS526_SK15_SMTR2_LFS, SamacSys_Parts:PTS526SK15SMTR2LFS, F.Cu at (444.9, -71.7)
- added S104: PTS526_SK15_SMTR2_LFS, SamacSys_Parts:PTS526SK15SMTR2LFS, F.Cu at (434.3, -63.4)
- added S201: EG1224 SPDT switch, SamacSys_Parts:EG1224, F.Cu at (236.7, 21.9)
- added U101: STM32L151C6Ux, Package_DFN_QFN:QFN-48-1EP_7x7mm_P0.5mm_EP5.6x5.6mm, F.Cu at (444.0, -62.9)
- added U201: APX810S05, Package_TO_SOT_SMD:SOT-23, F.Cu at (218.4, 44.1)
- added U202: 1043, SamacSys_Parts:1043, F.Cu at (156.1, 29.8)
- added U203: D1213A-02SM, Package_TO_SOT_SMD:SOT-23-5_HandSoldering, F.Cu at (213.0, 44.2)
- added U204: NE555P, Package_DIP:DIP-8_W7.62mm, F.Cu at (152.4, 59.2)
- added U601: LM4040DBZ-3, Package_TO_SOT_SMD:SOT-23, F.Cu at (259.6, -47.4)
- added U701: MC74VHC4052DR2G, Package_SO:SOIC-16_3.9x9.9mm_P1.27mm, F.Cu at (174.2, 82.7)
- added U702: MC74VHC4052DR2G, Package_SO:SOIC-16_3.9x9.9mm_P1.27mm, F.Cu at (174.2, 94.2)
- added U801: DIO6012BCST6, Package_TO_SOT_SMD:SOT-23-6_Handsoldering, F.Cu at (358.2, 4.95)
- added U901: MCP79412, Package_SO:TSSOP-8_4.4x3mm_P0.65mm, F.Cu at (345.0, -53.6)
- added Y901: 32.7680kHz, Crystal:Crystal_C38-LF_D3.0mm_L8.0mm_Vertical, F.Cu at (367.5, -73.3)
