File: STM32-Li-ion-charger-dischager-LCD.kicad_sch (KiCad schematic)
At the start: 35 parts

Commit message: soft
Parts:
- removed C? (x2): 1u, Capacitor_SMD:C_0603_1608Metric_Pad1.08x0.95mm_HandSolder, symbol Device:C_Small
- removed C?: 10n, Capacitor_SMD:C_0603_1608Metric_Pad1.08x0.95mm_HandSolder, symbol Device:C_Small
- removed FB?: HI1806T600R-10, SamacSys_Parts:BEADC4516X185N, symbol SamacSys_Parts:HI1806T600R-10
- removed U?: STM32L011K4Tx, Package_QFP:LQFP-32_7x7mm_P0.8mm, symbol MCU_ST_STM32L0:STM32L011K4Tx
- added C8, C9: 24P, Capacitor_SMD:C_0603_1608Metric_Pad1.08x0.95mm_HandSolder, symbol Device:C_Small
- added R? (x2): 10k, Resistor_SMD:R_0603_1608Metric_Pad0.98x0.95mm_HandSolder, symbol Device:R_Small
- added SW?: SW_SPDT, symbol Switch:SW_SPDT
- added Y1: 32k, symbol Device:Crystal_GND3_Small
- C1: renamed from C?; value 10n -> 4u7
- C3, C4: renamed from C?; value 10n -> 100n
- gave numbers to parts that had none: 27
Connections:
- net +3.3VA: now also U1.9 (VDDA)
- net +3V3: now also U1.24 (VDD), U1.36 (VDD), U1.48 (VDD), R?.1, SW?.3 (C)
- net D+: now also U1.33 (PA12)
- net D-: now also U1.32 (PA11)
- net GND: now also U1.23 (VSS), U1.35 (VSS), U1.47 (VSS), U1.49 (VSS), U1.8 (VSSA), C8.1, C9.1, SW?.1 (A), Y1.3
- net NRST: now also U1.7 (NRST), R?.2
- net UART_RX: now also U1.30 (PA9)
- net UART_TX: now also U1.31 (PA10)
- net osc_in: now also U1.5 (PH0)
- net osc_out: now also U1.6 (PH1)
- net MainClockOut: now reaches U1.29 (PA8)
- net at U1.3 (PC14): now also C8.2, Y1.1
- net at U1.4 (PC15): now also C9.2, Y1.2
- net BOOT0: now reaches U1.44 (BOOT0)
- net BOOT0: now also R?.2
- new net: R?.1, SW?.2 (B)
Other:
- note added: "HIGH FREQUENCY CLOCK"
- moved on the sheet: C1, C10, C11, C12, C13, C2, C3, C4, D1, FB2, J1, J2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

Commit message: t
Parts:
- removed J1, J2, J3: Conn_01x10, Connector_PinHeader_2.54mm:PinHeader_1x10_P2.54mm_Vertical, symbol Connector_Generic:Conn_01x10
Connections:
- net ADC4: no longer R1.2, U2.1 (K)
- new net V_ref: R1.2, U2.1 (K)
Other:
- added sheet ComponentTester (ComponentTester.kicad_sch)
- added sheet Display&SDcard (Display&SDcard.kicad_sch)
- note removed: "LCD"
- note removed: "SD card"
- moved on the sheet: R1, R?, SW?, U2

Commit message: t
Parts:
- removed R1: 1k, Resistor_SMD:R_0603_1608Metric_Pad0.98x0.95mm_HandSolder, symbol Device:R_Small
- removed U2: LM4040DBZ-3, Package_TO_SOT_SMD:SOT-23, symbol Reference_Voltage:LM4040DBZ-3
- gave numbers to parts that had none: 3
Other:
- added sheet EthernetLAN (EthernetLAN.kicad_sch)
- added sheet FanControl (FanControl.kicad_sch)
- sheet Display&SDcard ports: added SPI_CLK1, SPI_MISO1, SPI_MOSI1, SPI_ss1; removed none
- moved on the sheet: J4

Commit message: j
Other:
- sheet EthernetLAN renamed EthernetLAN+PoE
- sheet EthernetLAN+PoE ports: added SPI2_CLK, SPI2_MISO, SPI2_MOSI, SPI2_SS; removed none

Commit message: more work
Connections:
- net ADC1: now also U1.10 (PA0)
- net ADC2: now also U1.11 (PA1)
- net ADC3: now also U1.12 (PA2)
- net ADC4: now also U1.13 (PA3)
- net I2C_CLK: now also U1.42 (PB6)
- net I2C_SDA: now also U1.43 (PB7)
- net SPI_CLK: now also U1.26 (PB13)
- net SPI_MISO: now also U1.27 (PB14)
- net SPI_MOSI: now also U1.28 (PB15)
- net DAC1: now reaches U1.14 (PA4)
- net DAC2: now reaches U1.15 (PA5)
- net I2C2_CLK: now reaches U1.21 (PB10)
- net I2C2_SDA: now reaches U1.22 (PB11)
- net SPI2_CLK: now reaches U1.39 (PB3)
- net SPI2_MISO: now reaches U1.40 (PB4)
- net SPI2_MOSI: now reaches U1.41 (PB5)
- net UART_CTS: no longer names the net of J4.5 (Pin_5)
- net UART_RTS: no longer names the net of J4.6 (Pin_6)
Other:
- added sheet multiplexing+gpio_extenders (multiplexing+gpio_extenders.kicad_sch)
- sheet ComponentTester ports: added COMP1, COMP2, COMP3, COMP4, COMP5, COMP6; removed none
- sheet FanControl ports: added none; removed Thermistor

Commit message: h
Connections:
- net TOUCH_X: now reaches U1.16 (PA6)
- net TOUCH_Y: now reaches U1.17 (PA7)
Changed lines of the file:
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@@
+    (stroke (width 0) (type default) (color 0 0 0 0))
+  )
+  (wire (pts (xy 111.76 93.345) (xy 113.665 93.345))
     (stroke (width 0) (type default) (color 0 0 0 0))
   )
@@
   )
   (wire (pts (xy 66.04 31.115) (xy 52.07 31.115))
+    (stroke (width 0) (type default) (color 0 0 0 0))
+  )
+  (wire (pts (xy 111.76 90.805) (xy 113.665 90.805))
     (stroke (width 0) (type default) (color 0 0 0 0))
   )
@@
     )
   )
+  (global_label "TOUCH_X" (shape input) (at 113.665 90.805 0) (fields_autoplaced)
+    (effects (font (size 1.27 1.27)) (justify left))
+    (property "Intersheet References" "${INTERSHEET_REFS}" (id 0) (at 124.4843 90.8844 0)
+      (effects (font (size 1.27 1.27)) (justify left) hide)
+    )
+  )
   (global_label "SPI_CLK" (shape input) (at 52.07 170.815 180) (fields_autoplaced)
     (effects (font (size 1.27 1.27)) (justify right))
@@
     (property "Intersheet References" "${INTERSHEET_REFS}" (id 0) (at -32.2883 118.0306 0)
       (effects (font (size 1.27 1.27)) (justify right) hide)
+    )
+  )
+  (global_label "TOUCH_Y" (shape input) (at 113.665 93.345 0) (fields_autoplaced)
+    (effects (font (size 1.27 1.27)) (justify left))
+    (property "Intersheet References" "${INTERSHEET_REFS}" (id 0) (at 124.3633 93.4244 0)
+      (effects (font (size 1.27 1.27)) (justify left) hide)
     )
   )
@@
       (reference "IC4") (unit 1) (value "PEC12R-4230F-S0024") (footprint "PEC12R4230FS0024")
     )
+    (path "/9ca66431-4ae9-450d-a902-4ddfe318c744/1b0dc7d9-bdd8-4cc3-b800-a9d936cb284f"
+      (reference "IC?") (unit 1) (value "XRA1203IG24TR-F") (footprint "SOP65P640X120-24N")
+    )
     (path "/9ba7dc72-30ab-459c-b7f7-117aa274a468/f868776f-0ad2-4ffe-b528-607ce6660028"
       (reference "J1") (unit 1) (value "Conn_01x02") (footprint "Connector_PinHeader_2.54mm:PinHeader_1x02_P2.54mm_Vertical")
@@
       (reference "U11") (unit 1) (value "OPA188xxD") (footprint "Package_SO:SOIC-8_3.9x4.9mm_P1.27mm")
     )
-    (path "/9ca66431-4ae9-450d-a902-4ddfe318c744/4c726e0f-1585-43bc-ab71-e97533286e72"
-      (reference "U12") (unit 1) (value "CD4052B") (footprint "")
-    )
-    (path "/9ca66431-4ae9-450d-a902-4ddfe318c744/a8a0c780-e374-4b11-9834-fa797484e09e"
-      (reference "U13") (unit 1) (value "CD4052B") (footprint "")
+    (path "/9ca66431-4ae9-450d-a902-4ddfe318c744/6a9a2704-c264-456d-91fc-0c962ac61b47"
+      (reference "U?") (unit 1) (value "MC74VHC4052DR2G") (footprint "Package_SO:SOIC-16_3.9x9.9mm_P1.27mm")
+    )
+    (path "/9ca66431-4ae9-450d-a902-4ddfe318c744/71ebeb77-bc54-43d0-bad6-45405931d085"
+      (reference "U?") (unit 1) (value "MC74VHC4052DR2G") (footprint "Package_SO:SOIC-16_3.9x9.9mm_P1.27mm")
     )
     (path "/4849788e-5e45-4118-835e-f9b9ea5fb3c9"
