File: STM32-Li-ion-charger-dischager-LCD.kicad_sch (KiCad schematic)
At the start: 31 parts, among them J4 Conn_01x08, J5 USB_B_Mini, SW4 SW_SPDT, U1 STM32L151C6Ux, Y1 32k, Y2 32k

Commit message: n
Parts:
- added R? (x2): 10k, Resistor_SMD:R_0603_1608Metric_Pad0.98x0.95mm_HandSolder, symbol Device:R
Connections:
- net +3V3: now also R?.2, R?.2
- net I2C_CLK: now also R?.1
- net I2C_SDA: now also R?.1
Other:
- added sheet RTC (RTC.kicad_sch)
- note added: "OTHER"

Commit message: j
Parts:
- gave numbers to parts that had none: 2

Commit message: j
Other:
- removed sheet EthernetLAN+PoE

Commit message: h
Parts:
- added R107, R108, R109: 10k, Resistor_SMD:R_0603_1608Metric_Pad0.98x0.95mm_HandSolder, symbol Device:R
- renumbered C8 to C101, C9 to C102, C1 to C103, C10 to C104, C11 to C105, C2 to C106, C13 to C107, C3 to C108, C4 to C109, C12 to C110, C14 to C111, C15 to C112, C16 to C113, D1 to D101, FB2 to FB101, J4 to J101, J5 to J102, R1 to R101, R24 to R102, R2 to R103, R3 to R104, R4 to R105, R5 to R106, R74 to R110, R75 to R111, S4 to S101, S1 to S102, S2 to S103, S3 to S104, SW4 to SW101, U1 to U101, Y1 to Y101, Y2 to Y102
Connections:
- net +3V3: now also R107.2, R108.2, R109.2
- net SPI_CLK: now also R109.1
- net SPI_MISO: now also R108.1
- net SPI_MOSI: now also R107.1
Other:
- sheet multiplexing+gpio_extenders ports: added SCL, SDA; removed none
- moved on the sheet: J101
