File: EthernetLAN.kicad_sch (KiCad schematic)
At the start: 13 parts, among them J12 ARJM11C7-114-BA-EW2, U6 W5500

Commit message: j
Parts:
- added C? (x9): 100n, Capacitor_SMD:C_0603_1608Metric_Pad1.08x0.95mm_HandSolder, symbol Device:C_Small
- added C? (x2): 10u, Capacitor_SMD:C_0603_1608Metric_Pad1.08x0.95mm_HandSolder, symbol Device:C_Small
- added C?: 4u7, Capacitor_SMD:C_0603_1608Metric_Pad1.08x0.95mm_HandSolder, symbol Device:C_Small
- added D? (x2): LED_Small, LED_SMD:LED_0603_1608Metric_Pad1.05x0.95mm_HandSolder, symbol Device:LED_Small
- added R? (x4): 10K, Resistor_SMD:R_0603_1608Metric_Pad0.98x0.95mm_HandSolder, symbol Device:R_Small
- added R?: 12.4K, symbol Device:R_Small
- added R? (x2): 1k, Resistor_SMD:R_0603_1608Metric_Pad0.98x0.95mm_HandSolder, symbol Device:R_Small
- added R?: 10k, Resistor_SMD:R_0603_1608Metric_Pad0.98x0.95mm_HandSolder, symbol Device:R_Small
- added S?: PTS526_SK15_SMTR2_LFS, PTS526SK15SMTR2LFS, symbol SamacSys_Parts:PTS526_SK15_SMTR2_LFS
- added Y?: Crystal, symbol Device:Crystal
Connections:
- net +3V3: now also U6.28 (VDD), C?.1, C?.1, R?.1, R?.1, R?.1, R?.1, R?.1
- net GND: now also C?.1, C?.1, C?.1, C?.1, C?.1, C?.1, C?.1, C?.2, C?.2, C?.2, C?.2, C?.2, R?.2, R?.2, R?.2
- net at U6.10 (EXRES1): now also R?.1
- net +3.3VA: now reaches U6.11 (AVDD), U6.15 (AVDD), U6.17 (AVDD), U6.21 (AVDD), U6.4 (AVDD), U6.8 (AVDD)
- net +3.3VA: now also C?.1, C?.2, C?.2, C?.2, C?.2
- net at U6.20 (TOCAP): now also C?.1
- net at U6.22 (1V2O): now also C?.1
- net spd_led: now reaches U6.24 (SPDLED)
- net spd_led: now also D?.2 (A)
- net dup_led: now reaches U6.26 (DUPLED)
- net dup_led: now also D?.2 (A)
- net at U6.30 (XI/CLKIN): now also Y?.2
- net at U6.31 (XO): now also Y?.1
- net SPI2_SS: now reaches U6.32 (~{SCS})
- net SPI2_CLK: now reaches U6.33 (SCLK)
- net SPI2_MISO: now reaches U6.34 (MISO)
- net SPI2_MOSI: now reaches U6.35 (MOSI)
- net at U6.36 (~{INT}): now also R?.2
- net W5500_RST: now reaches U6.37 (~{RST})
- net W5500_RST: now also R?.2, S?.3 (NO_1), S?.4 (NO_2)
- net at U6.43 (PMODE2): now also R?.2
- net at U6.44 (PMODE1): now also R?.2
- net at U6.45 (PMODE0): now also R?.2
- new net: D?.1 (K), R?.1 (x2)
- new net: C?.2, S?.1 (COM_1), S?.2 (COM_2)
- no-connect marks 4 -> 7
Other:
- moved on the sheet: C30, C31, C32, C33, J12, R46, R47, R48, R49, R50, R51, R52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

Commit message: more work
Parts:
- added J14: Conn_02x07_Odd_Even, symbol Connector_Generic:Conn_02x07_Odd_Even
- gave numbers to parts that had none: 24
Connections:
- net VC1-: now reaches J12.1 (VC-_1)
- net VC1-: now also J14.1 (Pin_1), J14.2 (Pin_2)
- net VC2-: now reaches J12.2 (VC-_2)
- net VC2-: now also J14.10 (Pin_10), J14.9 (Pin_9)
- net VC1+: now reaches J12.6 (VC+_1)
- net VC1+: now also J14.5 (Pin_5), J14.6 (Pin_6)
- net VC2+: now reaches J12.7 (VC+_2)
- net VC2+: now also J14.13 (Pin_13), J14.14 (Pin_14)
- no-connect marks 7 -> 13
