File: BattDischarger.kicad_sch (KiCad schematic)
At the start: 27 parts

Commit message: soft
Parts:
- gave numbers to parts that had none: 27

Commit message: h
Parts:
- added C? (x2): 100n, Capacitor_SMD:C_0603_1608Metric_Pad1.08x0.95mm_HandSolder, symbol Device:C_Small
- added D?: D_Zener, symbol Device:D_Zener
- added D? (x2): D_Shockley, symbol Device:D_Shockley
- added Q?: Q_PMOS_DGS, symbol Device:Q_PMOS_DGS
- added R? (x6): 10k, Resistor_SMD:R_0603_1608Metric_Pad0.98x0.95mm_HandSolder, symbol Device:R_Small
- added R?: 47k, Resistor_SMD:R_0603_1608Metric_Pad0.98x0.95mm_HandSolder, symbol Device:R_Small
- added R?: 1k, Resistor_SMD:R_0603_1608Metric_Pad0.98x0.95mm_HandSolder, symbol Device:R_Small
- added U? (x3): LMH6609MA, Package_SO:SOIC-8_3.9x4.9mm_P1.27mm, symbol Amplifier_Operational:LMH6609MA
- R17: value 5m -> 10k
- R18: value 1m -> 10k
- R20: value 5m -> 47k
Connections:
- net GND: now also D?.2 (A), R?.2, U?.3 (+), U?.3 (+); no longer R18.2
- net V_batt3: now also D?.1 (K)
- net Measured_BATT+: now reaches BT3.1 (+), J9.2 (Pin_2), Q2.1 (D), R20.1
- net Measured_BATT+: now also R18.1
- net at JP2.1 (A): now also R18.2; no longer R18.1
- new net: R?.1, R?.1, R?.2, U?.2 (-)
- new net: D?.1 (K), D?.2 (A), U?.6
- new net: D?.2 (A), R?.1, R?.2
- new net: D?.1 (K), R?.1, R?.2, U?.2 (-)
- new net: R?.1, R?.2, R?.2, U?.6
- new net: R?.1, R?.2, U?.2 (-)
- new net: C?.1, C?.2
- new net: C?.2, R?.1
- new net ADC_internal_resistance: R?.1, U?.6
- new net DAC_SINE: R?.2
- new net Signal: C?.1, U?.3 (+)
Other:
- note added: "Capacity measurement section with CC set discharge or directly over R if we need/want"
- note added: "IRLZ44NPBF ? 1-2A Li-ion 4.2V so 3.2W at 1A ; 1.6W at 0.5A Pb acid 12-15V so 11W at 1A : 5-6W at 0.5A"
- note added: "Pre amplifier"
- note added: "precision full bridge rectifier"
- note added: "supercap fun"
- note removed: "IRLZ44NPBF ? 1-2A Li-ion 4.2V so 3.2W at 1A ; 1.6W at 0.5A Pb acid 12V so 11W at 1A : 5-6W at 0.5A"
- moved on the sheet: BT3, C24, C25, C26, C27, D7, HS1, J10, J8, J9, JP1, JP2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

Commit message: h
Parts:
- removed Q?: Q_PMOS_DGS, symbol Device:Q_PMOS_DGS
- added J?: Conn_01x02, symbol Connector_Generic:Conn_01x02
- added SW? (x2): SW_SPDT, symbol Switch:SW_SPDT
Connections:
- net Measured_BATT+: now also C?.1, C?.2
- net test_pwm: now also SW?.1 (A); no longer R13.1, R14.2
- net at C24.1, R14.1: now also SW?.1 (A); no longer U3.3 (+)
- new net: SW?.2 (B), U3.3 (+)
- new net: R13.1, R14.2, SW?.2 (B)
- new net test_DAC: SW?.3 (C)
Other:
- moved on the sheet: BT3, C24, C25, C26, C27, C?, D7, D?, HS1, J10, J8, J9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

Commit message: t
Parts:
- removed D? (x2): D_Shockley, symbol Device:D_Shockley
- removed R? (x6): 10k, Resistor_SMD:R_0603_1608Metric_Pad0.98x0.95mm_HandSolder, symbol Device:R_Small
- removed R?: 47k, Resistor_SMD:R_0603_1608Metric_Pad0.98x0.95mm_HandSolder, symbol Device:R_Small
- removed U? (x3): LMH6609MA, Package_SO:SOIC-8_3.9x4.9mm_P1.27mm, symbol Amplifier_Operational:LMH6609MA
Connections:
- net Signal renamed Signal_out
- net V_batt1 renamed BATT2+
- net V_batt2 renamed +BATT
- net V_batt3 renamed ADC5
- net load_I renamed ADC6_load
Other:
- note removed: "Pre amplifier"
- note removed: "precision full bridge rectifier"

Commit message: t
Parts:
- removed JP1: Jumper_2_Open, symbol Jumper:Jumper_2_Open
- removed R16: 10k, Resistor_SMD:R_0603_1608Metric_Pad0.98x0.95mm_HandSolder, symbol Device:R_Small
- removed R19: 50k, Resistor_SMD:R_0603_1608Metric_Pad0.98x0.95mm_HandSolder, symbol Device:R_Small
- removed SW?: SW_SPDT, symbol Switch:SW_SPDT
- added R29: 330, Resistor_THT:R_Axial_DIN0411_L9.9mm_D3.6mm_P7.62mm_Vertical, symbol Device:R_Small
- J1: renamed from J?; footprint (none) -> Connector_PinHeader_2.54mm:PinHeader_1x02_P2.54mm_Vertical
- gave numbers to parts that had none: 5
Connections:
- net GND: now also J1.1 (Pin_1)
- net test_DAC: now also J1.2 (Pin_2)
- net at C24.1, R14.1: now also U3.3 (+)
- net at SW3.1: now also R29.2; no longer D7.2 (A)
- net at Q2.2 (G), U4.1: now also U4.4 (-)
- new net: D7.2 (A), R29.1
Other:
- moved on the sheet: C24, J1, R13, R14, SW3, SW5

Commit message: more work
Parts:
- added D12: LED_Small, LED_SMD:LED_0603_1608Metric_Pad1.05x0.95mm_HandSolder, symbol Device:LED_Small
- added U8: OP179GRT, Package_TO_SOT_SMD:SOT-23-5, symbol Amplifier_Operational:OP179GRT
- R17: value 10k -> 5k
- R18: value 10k -> 1k
- R20: value 47k -> 10k
Connections:
- net GND: now also R18.2, U8.5 (V-)
- net Measured_BATT+: no longer R18.1
- net at JP2.1 (A): now also R18.1; no longer R18.2
- net ADC5 renamed measured_batt_v
- net measured_batt_v: now also U8.3 (+)
- net ADC6_load renamed measured_batt_I
- new net divider_state: D12.2 (A), U8.1
Other:
- moved on the sheet: BT3, C24, C25, C26, C27, C28, C7, D7, D8, HS1, J1, J10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

Commit message: j
Parts:
- removed SW3: RA12131100, symbol My_custom_lib:RA12131100
- added SW?: RA12131100, Z_mycustom_footprint_lib:RA12131100, symbol My_custom_lib:RA12131100
Connections:
- net VBUS: now also SW?.2
- net at R29.2: now also SW?.1
Other:
- moved on the sheet: C26, C27, D7, J10, R22, R23, R29
