File: BattDischarger.kicad_sch (KiCad schematic)
At the start: 33 parts, among them J1 Conn_01x02, J10 Conn_01x02, J8 Conn_01x03, J9 Conn_01x02, Q2 Q_NMOS_DGS, SW5 SW_SPDT, U3 OP179GRT, U4 OP179GRT, U8 OP179GRT

Commit message: h
Parts:
- removed C26, C27: 3.3, Capacitor_THT:CP_Radial_D8.0mm_P3.50mm, symbol Device:C_Polarized_Small
- removed D7: D_Shockley, Diode_THT:D_A-405_P12.70mm_Horizontal, symbol Device:D_Shockley
- removed J10: Conn_01x02, Resistor_THT:R_Axial_DIN0309_L9.0mm_D3.2mm_P5.08mm_Vertical, symbol Connector_Generic:Conn_01x02
- removed R22, R23: 1M, Resistor_THT:R_Axial_DIN0411_L9.9mm_D3.6mm_P7.62mm_Vertical, symbol Device:R_Small
- removed R29: 330, Resistor_THT:R_Axial_DIN0411_L9.9mm_D3.6mm_P7.62mm_Vertical, symbol Device:R_Small
- removed SW?: RA12131100, Z_mycustom_footprint_lib:RA12131100, symbol My_custom_lib:RA12131100
- removed U3, U4, U8: OP179GRT, Package_TO_SOT_SMD:SOT-23-5, symbol Amplifier_Operational:OP179GRT
- added U301: (no value), symbol Amplifier_Operational:LM324A
- renumbered BT3 to BT301, C24 to C301, C25 to C302, C7 to C303, C28 to C304, D8 to D301, D12 to D302, HS1 to HS301, J1 to J301, J8 to J302, J9 to J303, JP2 to JP301, Q2 to Q301, R13 to R301, R14 to R302, R15 to R303, R17 to R304, R18 to R305, R20 to R306, R21 to R307, R30 to R308, SW5 to SW301
Connections:
- net divider_state: now also U301.8
- net measured_batt_I: now also U301.2 (-)
- net measured_batt_v: now also U301.10 (+)
- net at C301.1, R302.1: now also U301.3 (+)
- net at C302.2, R303.1: now also U301.5 (+)
- net at R303.2: now also U301.1
- net at Q301.2 (G): now also U301.6 (-), U301.7
- new net +12V: U301.4 (V+)
- new net -12V: U301.11 (V-)
Other:
- note removed: "supercap fun"
