File: ComponentTester.kicad_sch (KiCad schematic)
At the start: 15 parts

Commit message: t
Parts:
- gave numbers to parts that had none: 15
Changed lines of the file:
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@@
   (symbol (lib_id "power:GND") (at 160.655 65.405 0) (unit 1)
     (in_bom yes) (on_board yes) (fields_autoplaced)
-    (property "Reference" "#PWR?" (id 0) (at 160.655 71.755 0)
+    (property "Reference" "#PWR014" (id 0) (at 160.655 71.755 0)
       (effects (font (size 1.27 1.27)) hide)
     )
@@
   (symbol (lib_id "Device:R_Small") (at 64.135 78.74 90) (unit 1)
     (in_bom yes) (on_board yes) (fields_autoplaced)
-    (property "Reference" "R?" (id 0) (at 64.135 72.39 90))
+    (property "Reference" "R35" (id 0) (at 64.135 72.39 90))
     (property "Value" "680" (id 1) (at 64.135 74.93 90))
     (property "Footprint" "" (id 2) (at 64.135 78.74 0)
@@
   (symbol (lib_id "Connector_Generic:Conn_01x02") (at 151.13 65.405 180) (unit 1)
     (in_bom yes) (on_board yes)
-    (property "Reference" "J?" (id 0) (at 150.495 72.39 0))
+    (property "Reference" "J11" (id 0) (at 150.495 72.39 0))
     (property "Value" "Conn_01x02" (id 1) (at 151.13 69.85 0))
     (property "Footprint" "" (id 2) (at 151.13 65.405 0)
@@
   (symbol (lib_id "power:+3.3V") (at 156.845 42.545 90) (unit 1)
     (in_bom yes) (on_board yes) (fields_autoplaced)
-    (property "Reference" "#PWR?" (id 0) (at 160.655 42.545 0)
+    (property "Reference" "#PWR012" (id 0) (at 160.655 42.545 0)
       (effects (font (size 1.27 1.27)) hide)
     )
@@
   (symbol (lib_id "Device:R_Small") (at 64.135 66.04 90) (unit 1)
     (in_bom yes) (on_board yes)
-    (property "Reference" "R?" (id 0) (at 64.135 69.85 90))
+    (property "Reference" "R34" (id 0) (at 64.135 69.85 90))
     (property "Value" "470k" (id 1) (at 64.135 67.945 90))
     (property "Footprint" "" (id 2) (at 64.135 66.04 0)
@@
   (symbol (lib_id "power:GND") (at 186.69 42.545 90) (unit 1)
     (in_bom yes) (on_board yes) (fields_autoplaced)
-    (property "Reference" "#PWR?" (id 0) (at 193.04 42.545 0)
+    (property "Reference" "#PWR015" (id 0) (at 193.04 42.545 0)
       (effects (font (size 1.27 1.27)) hide)
     )
@@
   (symbol (lib_id "Device:R_Small") (at 64.135 81.915 90) (unit 1)
     (in_bom yes) (on_board yes)
-    (property "Reference" "R?" (id 0) (at 64.135 85.725 90))
+    (property "Reference" "R36" (id 0) (at 64.135 85.725 90))
     (property "Value" "470k" (id 1) (at 64.135 83.82 90))
     (property "Footprint" "" (id 2) (at 64.135 81.915 0)
@@
   (symbol (lib_id "Device:R_Small") (at 182.245 42.545 90) (mirror x) (unit 1)
     (in_bom yes) (on_board yes)
-    (property "Reference" "R?" (id 0) (at 180.975 47.625 0)
+    (property "Reference" "R38" (id 0) (at 180.975 47.625 0)
       (effects (font (size 1.27 1.27)) (justify right))
     )
@@
     (pin "2")
   )
+  (symbol (lib_id "power:+12V") (at 209.55 48.26 0) (unit 1)
+    (in_bom yes) (on_board yes) (fields_autoplaced)
+    (property "Reference" "#PWR017" (id 0) (at 209.55 52.07 0)
+      (effects (font (size 1.27 1.27)) hide)
+    )
+    (property "Value" "+12V" (id 1) (at 209.55 43.18 0))
+    (property "Footprint" "" (id 2) (at 209.55 48.26 0)
+      (effects (font (size 1.27 1.27)) hide)
+    )
+    (property "Datasheet" "" (id 3) (at 209.55 48.26 0)
+      (effects (font (size 1.27 1.27)) hide)
+    )
+    (pin "1")
+  )
   (symbol (lib_id "Connector_Generic:Conn_01x02") (at 151.13 59.69 180) (unit 1)
     (in_bom yes) (on_board yes) (fields_autoplaced)
-    (property "Reference" "J?" (id 0) (at 151.13 50.8 0))
+    (property "Reference" "J3" (id 0) (at 151.13 50.8 0))
     (property "Value" "Conn_01x02" (id 1) (at 151.13 53.34 0))
     (property "Footprint" "" (id 2) (at 151.13 59.69 0)
@@
   (symbol (lib_id "Device:C_Small") (at 165.735 60.96 90) (mirror x) (unit 1)
     (in_bom yes) (on_board yes)
-    (property "Reference" "C?" (id 0) (at 167.005 63.5 0)
+    (property "Reference" "C29" (id 0) (at 167.005 63.5 0)
       (effects (font (size 1.27 1.27)) (justify left))
     )
@@
   (symbol (lib_id "Device:R_Small") (at 64.135 46.99 90) (unit 1)
     (in_bom yes) (on_board yes) (fields_autoplaced)
-    (property "Reference" "R?" (id 0) (at 64.135 40.64 90))
+    (property "Reference" "R31" (id 0) (at 64.135 40.64 90))
     (property "Value" "680" (id 1) (at 64.135 43.18 90))
     (property "Footprint" "" (id 2) (at 64.135 46.99 0)
@@
   (symbol (lib_id "Connector_Generic:Conn_01x03") (at 75.565 30.48 90) (unit 1)
     (in_bom yes) (on_board yes) (fields_autoplaced)
-    (property "Reference" "J?" (id 0) (at 81.28 29.2099 90)
+    (property "Reference" "J2" (id 0) (at 81.28 29.2099 90)
       (effects (font (size 1.27 1.27)) (justify right))
     )
@@
     (pin "3")
   )
+  (symbol (lib_id "power:-12V") (at 207.01 87.63 0) (unit 1)
+    (in_bom yes) (on_board yes) (fields_autoplaced)
+    (property "Reference" "#PWR016" (id 0) (at 207.01 85.09 0)
+      (effects (font (size 1.27 1.27)) hide)
+    )
+    (property "Value" "-12V" (id 1) (at 207.01 82.55 0))
+    (property "Footprint" "" (id 2) (at 207.01 87.63 0)
+      (effects (font (size 1.27 1.27)) hide)
+    )
+    (property "Datasheet" "" (id 3) (at 207.01 87.63 0)
+      (effects (font (size 1.27 1.27)) hide)
+    )
+    (pin "1")
+  )
   (symbol (lib_id "power:GND") (at 160.655 57.15 180) (unit 1)
     (in_bom yes) (on_board yes) (fields_autoplaced)
-    (property "Reference" "#PWR?" (id 0) (at 160.655 50.8 0)
+    (property "Reference" "#PWR013" (id 0) (at 160.655 50.8 0)
       (effects (font (size 1.27 1.27)) hide)
     )
@@
   (symbol (lib_id "Device:R_Small") (at 64.135 50.165 90) (unit 1)
     (in_bom yes) (on_board yes)
-    (property "Reference" "R?" (id 0) (at 64.135 53.975 90))
+    (property "Reference" "R32" (id 0) (at 64.135 53.975 90))
     (property "Value" "470k" (id 1) (at 64.135 52.07 90))
     (property "Footprint" "" (id 2) (at 64.135 50.165 0)
@@
   (symbol (lib_id "Device:R_Potentiometer") (at 173.355 42.545 270) (unit 1)
     (in_bom yes) (on_board yes)
-    (property "Reference" "RV?" (id 0) (at 172.847 35.687 90))
+    (property "Reference" "RV3" (id 0) (at 172.847 35.687 90))
     (property "Value" "47k" (id 1) (at 174.879 38.735 90))
     (property "Footprint" "Z_mycustom_footprint_lib:2002102255" (id 2) (at 173.355 42.545 0)
@@
   (symbol (lib_id "Device:R_Small") (at 64.135 62.865 90) (unit 1)
     (in_bom yes) (on_board yes) (fields_autoplaced)
-    (property "Reference" "R?" (id 0) (at 64.135 56.515 90))
+    (property "Reference" "R33" (id 0) (at 64.135 56.515 90))
     (property "Value" "680" (id 1) (at 64.135 59.055 90))
     (property "Footprint" "" (id 2) (at 64.135 62.865 0)
@@
   (symbol (lib_id "Device:R_Small") (at 182.245 60.96 270) (mirror x) (unit 1)
     (in_bom yes) (on_board yes)
-    (property "Reference" "R?" (id 0) (at 183.515 55.88 0)
+    (property "Reference" "R39" (id 0) (at 183.515 55.88 0)
       (effects (font (size 1.27 1.27)) (justify right))
     )
@@
   (symbol (lib_id "Device:R_Small") (at 162.56 42.545 90) (mirror x) (unit 1)
     (in_bom yes) (on_board yes)
-    (property "Reference" "R?" (id 0) (at 161.29 47.625 0)
+    (property "Reference" "R37" (id 0) (at 161.29 47.625 0)
       (effects (font (size 1.27 1.27)) (justify right))
     )
@@
   (symbol (lib_id "Amplifier_Operational:OPA188xxD") (at 212.725 63.5 0) (unit 1)
     (in_bom yes) (on_board yes) (fields_autoplaced)
-    (property "Reference" "U?" (id 0) (at 224.155 58.801 0))
+    (property "Reference" "U2" (id 0) (at 224.155 58.801 0))
     (property "Value" "OPA188xxD" (id 1) (at 224.155 61.341 0))
     (property "Footprint" "Package_SO:SOIC-8_3.9x4.9mm_P1.27mm" (id 2) (at 210.185 68.58 0)

Commit message: more work
Parts:
- added C50, C51, C52: 1u, Capacitor_SMD:C_0603_1608Metric_Pad1.08x0.95mm_HandSolder, symbol Device:C_Small
- added J15, J16, J17, J18, J19, J20: Conn_01x02, symbol Connector_Generic:Conn_01x02
- added R59, R60, R61, R62, R63, R64, R65, R66, R67: 50k, Resistor_SMD:R_0603_1608Metric_Pad0.98x0.95mm_HandSolder, symbol Device:R_Small
- added RV4, RV5, RV6: 47k, Z_mycustom_footprint_lib:2002102255, symbol Device:R_Potentiometer
- added U10, U11, U9: OPA188xxD, Package_SO:SOIC-8_3.9x4.9mm_P1.27mm, symbol Amplifier_Operational:OPA188xxD
Connections:
- net +3V3: now also R59.1, R60.1, R61.1
- net GND: now also J15.2 (Pin_2), J16.1 (Pin_1), J17.2 (Pin_2), J18.1 (Pin_1), J19.2 (Pin_2), J20.1 (Pin_1), R62.2, R64.2, R66.2
- net COMP5: now reaches R35.1
- net COMP4: now reaches R34.1
- net COMP6: now reaches R36.1
- net COMP1: now reaches R31.1
- net COMP2: now reaches R32.1
- net COMP3: now reaches R33.1
- net ADC1 renamed component1
- net ADC2 renamed component2
- net ADC3 renamed component3
- net ADC4 renamed scope1
- new net: R60.2, RV5.3
- new net: R66.1, RV6.1
- new net: C52.1, J19.1 (Pin_1), J20.2 (Pin_2)
- new net: R67.1, U11.3 (+)
- new net: C52.2, R67.2, RV6.2
- new net: R64.1, RV5.1
- new net: R59.2, RV4.3
- new net: R61.2, RV6.3
- new net: C50.1, J15.1 (Pin_1), J16.2 (Pin_2)
- new net: R65.1, U10.3 (+)
- new net: C51.2, R65.2, RV5.2
- new net: R62.1, RV4.1
- new net: C51.1, J17.1 (Pin_1), J18.2 (Pin_2)
- new net: C50.2, R63.2, RV4.2
- new net: U10.2 (-), U10.6
- new net: U9.2 (-), U9.6
- new net: R63.1, U9.3 (+)
- new net: U11.2 (-), U11.6
Other:
- moved on the sheet: C29, J11, J2, J3, R31, R32, R33, R34, R35, R36, R37, R38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

Commit message: h
Parts:
- removed R37, R38, R59, R60, R61, R62, R64, R66: 50k, Resistor_SMD:R_0603_1608Metric_Pad0.98x0.95mm_HandSolder, symbol Device:R_Small
- removed U10, U11, U2, U9: OPA188xxD, Package_SO:SOIC-8_3.9x4.9mm_P1.27mm, symbol Amplifier_Operational:OPA188xxD
- added U401: (no value), symbol Amplifier_Operational:LM324A
- renumbered C50 to C401, C51 to C402, C29 to C403, C52 to C404, J15 to J401, J16 to J402, J17 to J403, J18 to J404, J3 to J405, J11 to J406, J19 to J407, J20 to J408, J2 to J409, R63 to R401, R65 to R402, R39 to R403, R67 to R404, R31 to R405, R32 to R406, R33 to R407, R34 to R408, R35 to R409, R36 to R410, RV4 to RV401, RV5 to RV402, RV3 to RV403, RV6 to RV404
Connections:
- net +12V: now also U401.4 (V+)
- net +3V3: now also RV401.3, RV402.3, RV403.3, RV404.3
- net -12V: now also U401.11 (V-)
- net GND: now also RV401.1, RV402.1, RV403.1, RV404.1
- net scope1: now also U401.1, U401.2 (-)
- net scope2: now also U401.6 (-), U401.7
- net scope3: now also U401.8, U401.9 (-)
- net scope4: now also U401.13 (-), U401.14
- net at R404.1: now also U401.10 (+)
- net at R402.1: now also U401.12 (+)
- net at R401.1: now also U401.5 (+)
- net at R403.1: now also U401.3 (+)
Other:
- moved on the sheet: C401, C402, C403, C404, J401, J402, J403, J404, J405, J406, J407, J408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
