File: Display&SDcard.kicad_sch (KiCad schematic)
At the start: 0 parts

Commit message: t
Parts:
- added B1: ARDUINO_UNO_R3_SHIELDBASIC, UNO_R3_SHIELD, symbol SparkFun-Boards:ARDUINO_UNO_R3_SHIELDBASIC
Changed lines of the file:
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@@
     )
+  )
+  (hierarchical_label "SPI_CLK1" (shape input) (at 247.015 113.665 0)
+    (effects (font (size 1.27 1.27)) (justify left))
+  )
+  (hierarchical_label "SPI_MISO1" (shape input) (at 247.65 107.315 0)
+    (effects (font (size 1.27 1.27)) (justify left))
+  )
+  (hierarchical_label "SPI_ss1" (shape input) (at 247.65 98.425 0)
+    (effects (font (size 1.27 1.27)) (justify left))
+  )
+  (hierarchical_label "SPI_MOSI1" (shape input) (at 247.015 103.505 0)
+    (effects (font (size 1.27 1.27)) (justify left))
   )
   (symbol (lib_id "power:GND") (at 212.725 74.295 0) (mirror y) (unit 1)
     (in_bom yes) (on_board yes) (fields_autoplaced)
-    (property "Reference" "#PWR?" (id 0) (at 212.725 80.645 0)
+    (property "Reference" "#PWR020" (id 0) (at 212.725 80.645 0)
       (effects (font (size 1.27 1.27)) hide)
     )
@@
     (pin "1")
   )
+  (symbol (lib_id "SparkFun-Boards:ARDUINO_UNO_R3_SHIELDBASIC") (at 136.525 87.63 0) (unit 1)
+    (in_bom yes) (on_board yes) (fields_autoplaced)
+    (property "Reference" "B1" (id 0) (at 136.525 59.69 0)
+      (effects (font (size 1.143 1.143)))
+    )
+    (property "Value" "ARDUINO_UNO_R3_SHIELDBASIC" (id 1) (at 136.525 62.23 0)
+      (effects (font (size 1.143 1.143)))
+    )
+    (property "Footprint" "UNO_R3_SHIELD" (id 2) (at 136.525 63.5 0)
+      (effects (font (size 0.508 0.508)) hide)
+    )
+    (property "Datasheet" "" (id 3) (at 136.525 87.63 0)
+      (effects (font (size 1.27 1.27)) hide)
+    )
+    (property "Field4" "XXX-00000" (id 4) (at 136.525 66.04 0)
+      (effects (font (size 1.524 1.524)))
+    )
+    (pin "3.3V")
+    (pin "5V")
+    (pin "A0")
+    (pin "A1")
+    (pin "A2")
+    (pin "A3")
+    (pin "A4")
+    (pin "A5")
+    (pin "AREF")
+    (pin "D10")
+    (pin "D11")
+    (pin "D12")
+    (pin "D13")
+    (pin "D2")
+    (pin "D3")
+    (pin "D4")
+    (pin "D5")
+    (pin "D6")
+    (pin "D7")
+    (pin "D8")
+    (pin "D9")
+    (pin "GND@")
+    (pin "GND@")
+    (pin "GND@")
+    (pin "IORE")
+    (pin "RES")
+    (pin "RX")
+    (pin "SCL")
+    (pin "SDA")
+    (pin "TX")
+    (pin "VIN")
+  )
   (symbol (lib_id "power:+3.3V") (at 216.535 66.675 0) (mirror y) (unit 1)
     (in_bom yes) (on_board yes) (fields_autoplaced)
-    (property "Reference" "#PWR?" (id 0) (at 216.535 70.485 0)
+    (property "Reference" "#PWR021" (id 0) (at 216.535 70.485 0)
       (effects (font (size 1.27 1.27)) hide)
     )
@@
   (symbol (lib_id "power:+3.3V") (at 207.01 99.06 0) (mirror y) (unit 1)
     (in_bom yes) (on_board yes) (fields_autoplaced)
-    (property "Reference" "#PWR?" (id 0) (at 207.01 102.87 0)
+    (property "Reference" "#PWR019" (id 0) (at 207.01 102.87 0)
       (effects (font (size 1.27 1.27)) hide)
     )
@@
   (symbol (lib_id "power:GND") (at 203.2 106.68 0) (mirror y) (unit 1)
     (in_bom yes) (on_board yes) (fields_autoplaced)
-    (property "Reference" "#PWR?" (id 0) (at 203.2 113.03 0)
+    (property "Reference" "#PWR018" (id 0) (at 203.2 113.03 0)
       (effects (font (size 1.27 1.27)) hide)
     )

Commit message: more work
Connections:
- net +3V3: now also B1.3.3V
- net GND: now also B1.GND@ (GND)
- net SPI_CLK1: now also B1.D13
- net SPI_MISO1: now also B1.D11 (*D11)
- net SPI_MOSI1: now also B1.D12
- net LCD_CONTROL: now reaches B1.A0
- net TOUCH_Y: now reaches B1.A1
- net TOUCH_X: now reaches B1.A2
- net LCD_CS: now reaches B1.A3
- net LCD_RST: now reaches B1.A4
- net SPI_SS1: now reaches B1.D10 (*D10)
- net LCD_D2: now reaches B1.D2
- net LCD_D3: now reaches B1.D3 (*D3)
- net LCD_D4: now reaches B1.D4
- net LCD_D5: now reaches B1.D5 (*D5)
- net LCD_D6: now reaches B1.D6 (*D6)
- net LCD_D7: now reaches B1.D7
- net LCD_D0: now reaches B1.D8
- net LCD_D1: now reaches B1.D9 (*D9)
- no-connect marks 0 -> 10
Other:
- note removed: "LCD"
- note removed: "SD card"

Commit message: h
Parts:
- renumbered B1 to B501
Changed lines of the file:
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@@
   (symbol (lib_id "power:GND") (at 123.825 114.3 0) (mirror y) (unit 1)
     (in_bom yes) (on_board yes) (fields_autoplaced)
-    (property "Reference" "#PWR020" (id 0) (at 123.825 120.65 0)
+    (property "Reference" "#PWR0502" (id 0) (at 123.825 120.65 0)
       (effects (font (size 1.27 1.27)) hide)
     )
@@
   (symbol (lib_id "SparkFun-Boards:ARDUINO_UNO_R3_SHIELDBASIC") (at 136.525 87.63 0) (unit 1)
     (in_bom yes) (on_board yes) (fields_autoplaced)
-    (property "Reference" "B1" (id 0) (at 136.525 59.69 0)
+    (property "Reference" "B501" (id 0) (at 136.525 59.69 0)
       (effects (font (size 1.143 1.143)))
     )
@@
   (symbol (lib_id "power:+3.3V") (at 119.38 100.33 90) (mirror x) (unit 1)
     (in_bom yes) (on_board yes) (fields_autoplaced)
-    (property "Reference" "#PWR019" (id 0) (at 123.19 100.33 0)
+    (property "Reference" "#PWR0501" (id 0) (at 123.19 100.33 0)
       (effects (font (size 1.27 1.27)) hide)
     )
