File: FanControl.kicad_sch (KiCad schematic)
At the start: 12 parts, among them M1 Fan_3pin, Q4 Q_PMOS_DGS, Q5 Q_NMOS_DGS, U5 LM4040DBZ-3

Commit message: more work
Parts:
- added R68, R69, R70, R71, R72, R73, R? (x4): 10k, Resistor_SMD:R_0603_1608Metric_Pad0.98x0.95mm_HandSolder, symbol Device:R_Small
Connections:
- net +3V3: now also R68.1, R69.1, R70.1, R71.1, R72.1, R73.1, R?.1, R?.1, R?.1, R?.1
- net Thermistor renamed thermistor
- new net I2C2_CLK: R?.2
- new net I2C2_SDA: R?.2
- new net I2C_CLK: R?.2
- new net I2C_SDA: R?.2
- new net SPI2_CLK: R71.2
- new net SPI2_MISO: R72.2
- new net SPI2_MOSI: R73.2
- new net SPI_CLK: R70.2
- new net SPI_MISO: R69.2
- new net SPI_MOSI: R68.2

Commit message: j
Parts:
- gave numbers to parts that had none: 4
Changed lines of the file:
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@@
   (symbol (lib_id "Device:R_Small") (at 38.735 157.48 270) (unit 1)
     (in_bom yes) (on_board yes) (fields_autoplaced)
-    (property "Reference" "R?" (id 0) (at 38.735 151.765 90))
+    (property "Reference" "R84" (id 0) (at 38.735 151.765 90))
     (property "Value" "10k" (id 1) (at 38.735 154.305 90))
     (property "Footprint" "Resistor_SMD:R_0603_1608Metric_Pad0.98x0.95mm_HandSolder" (id 2) (at 38.735 157.48 0)
@@
   (symbol (lib_id "Device:R_Small") (at 38.735 149.86 270) (unit 1)
     (in_bom yes) (on_board yes) (fields_autoplaced)
-    (property "Reference" "R?" (id 0) (at 38.735 144.145 90))
+    (property "Reference" "R81" (id 0) (at 38.735 144.145 90))
     (property "Value" "10k" (id 1) (at 38.735 146.685 90))
     (property "Footprint" "Resistor_SMD:R_0603_1608Metric_Pad0.98x0.95mm_HandSolder" (id 2) (at 38.735 149.86 0)
@@
   (symbol (lib_id "Device:R_Small") (at 38.735 154.94 270) (unit 1)
     (in_bom yes) (on_board yes) (fields_autoplaced)
-    (property "Reference" "R?" (id 0) (at 38.735 149.225 90))
+    (property "Reference" "R83" (id 0) (at 38.735 149.225 90))
     (property "Value" "10k" (id 1) (at 38.735 151.765 90))
     (property "Footprint" "Resistor_SMD:R_0603_1608Metric_Pad0.98x0.95mm_HandSolder" (id 2) (at 38.735 154.94 0)
@@
   (symbol (lib_id "Device:R_Small") (at 38.735 152.4 270) (unit 1)
     (in_bom yes) (on_board yes) (fields_autoplaced)
-    (property "Reference" "R?" (id 0) (at 38.735 146.685 90))
+    (property "Reference" "R82" (id 0) (at 38.735 146.685 90))
     (property "Value" "10k" (id 1) (at 38.735 149.225 90))
     (property "Footprint" "Resistor_SMD:R_0603_1608Metric_Pad0.98x0.95mm_HandSolder" (id 2) (at 38.735 152.4 0)

Commit message: h
Parts:
- removed R68, R69, R70, R71, R72, R73, R81, R82, R83, R84: 10k, Resistor_SMD:R_0603_1608Metric_Pad0.98x0.95mm_HandSolder, symbol Device:R_Small
- renumbered D9 to D601, M1 to M601, Q4 to Q601, Q5 to Q602, R40 to R601, R41 to R602, R42 to R603, R43 to R604, R44 to R605, R45 to R606, TH1 to TH601, U5 to U601
