File: PowerManagement.kicad_sch (KiCad schematic)
At the start: 32 parts

Commit message: soft
Parts:
- added C?: 10n, Capacitor_SMD:C_0603_1608Metric_Pad1.08x0.95mm_HandSolder, symbol Device:C_Small
- added C?: 1u, Capacitor_SMD:C_0603_1608Metric_Pad1.08x0.95mm_HandSolder, symbol Device:C_Small
- added FB?: HI1806T600R-10, SamacSys_Parts:BEADC4516X185N, symbol SamacSys_Parts:HI1806T600R-10
- gave numbers to parts that had none: 32
Connections:
- net +3V3: now also FB?.1
- net GND: now also C?.2, C?.2
- new net +3.3VA: C?.1, C?.1, FB?.2

Commit message: t
Parts:
- added Q?: Q_PMOS_DGS, symbol Device:Q_PMOS_DGS
- added R? (x4): 50k, Resistor_SMD:R_0603_1608Metric_Pad0.98x0.95mm_HandSolder, symbol Device:R_Small
Connections:
- net +5V: now also Q?.2 (G)
- net +BATT: now also R?.1
- net +VDC: now also Q?.3 (S); no longer Q1.1 (D)
- net GND: now also R?.2, R?.2
- net V_batt2 renamed BATT2+
- net BATT2+: now also R?.1
- new net: Q1.1 (D), Q?.1 (D)
- new net ADC6: R?.1, R?.2
- new net ADC7: R?.1, R?.2
Other:
- moved on the sheet: D6, Q1, R6

Commit message: t
Parts:
- added C? (x2): 4.7u, Capacitor_SMD:C_0603_1608Metric_Pad1.08x0.95mm_HandSolder, symbol Device:C_Small
- added D? (x2): DIODE, symbol Simulation_SPICE:DIODE
- gave numbers to parts that had none: 8
Connections:
- net GND: now also C?.2, D?.2 (K)
- new net: C?.2, D?.1 (A), D?.2 (K)
- new net -12V: C?.1, D?.1 (A)
Other:
- note added: "large pwm as in peack to peack"

Commit message: more work
Parts:
- added C34, C35: 100n, Capacitor_SMD:C_0603_1608Metric_Pad1.08x0.95mm_HandSolder, symbol Device:C_Small
- added D15: D_Shockley, Diode_THT:D_A-405_P12.70mm_Horizontal, symbol Device:D_Shockley
- added J13: Conn_01x02, Connector_PinHeader_2.54mm:PinHeader_1x02_P2.54mm_Vertical, symbol Connector_Generic:Conn_01x02
- added RTHT1: 1k, symbol Device:R_Small
- added RTHT2: 4.7k, symbol Device:R_Small
- added U7: NE555P, Package_DIP:DIP-8_W7.62mm, symbol Timer:NE555P
- gave numbers to parts that had none: 4
Connections:
- net +VDC: now also D15.1 (K)
- net GND: now also C34.1, C35.1, J13.1 (Pin_1), U7.1 (GND)
- net at C36.1: now also U7.3 (Q)
- net ADC6 renamed bat1_v
- net ADC7 renamed bat2_v
- new net: D15.2 (A), J13.2 (Pin_2)
- new net: C34.2, U7.5 (CV)
- new net: C35.2, RTHT2.2, U7.2 (TR), U7.6 (THR)
- new net: RTHT1.2, RTHT2.1, U7.7 (DIS)
- new net +12V: RTHT1.1, U7.4 (R), U7.8 (VCC)
Other:
- moved on the sheet: C36, C37, C5, C6, D10, D11, FB1

Commit message: n
Parts:
- added BT?: Battery, symbol Device:Battery
- added C? (x2): 1u, Capacitor_SMD:C_0805_2012Metric_Pad1.18x1.45mm_HandSolder, symbol Device:C_Small
- added D? (x3): LED_Small Green, LED_SMD:LED_0603_1608Metric_Pad1.05x0.95mm_HandSolder, symbol Device:LED_Small
- added D?: D_Shockley, Diode_THT:D_DO-15_P15.24mm_Horizontal, symbol Device:D_Shockley
- added F?: Polyfuse_Small, Fuse:Fuse_1812_4532Metric_Pad1.30x3.40mm_HandSolder, symbol Device:Polyfuse_Small
- added FB?: HI1806T600R-10, SamacSys_Parts:BEADC4516X185N, symbol SamacSys_Parts:HI1806T600R-10
- added IC?: AP2112M-3.3TRG1, SamacSys_Parts:SOIC127P600X170-8N, symbol SamacSys_Parts:AP2112M-3.3TRG1
- added J?: Conn_01x03, Connector_PinHeader_2.54mm:PinHeader_1x03_P2.54mm_Vertical, symbol Connector_Generic:Conn_01x03
- added J?: USB_B_Mini, Connector_USB:USB_Mini-B_Lumberg_2486_01_Horizontal, symbol Connector:USB_B_Mini
- added J?: Conn_01x02_Male, Connector_PinHeader_2.54mm:PinHeader_1x02_P2.54mm_Vertical, symbol Connector:Conn_01x02_Male
- added Q?: DMG9933USD-13, SamacSys_Parts:SOIC127P600X175-8N, symbol SamacSys_Parts:DMG9933USD-13
- added R? (x2): 330, Resistor_SMD:R_0603_1608Metric_Pad0.98x0.95mm_HandSolder, symbol Device:R
- added R?: 10k, Resistor_SMD:R_0603_1608Metric_Pad0.98x0.95mm_HandSolder, symbol Device:R
- added R?: 10k+ pullup, Resistor_SMD:R_0603_1608Metric_Pad0.98x0.95mm_HandSolder, symbol Device:R
- added R?: 4.7k, Resistor_THT:R_Axial_DIN0204_L3.6mm_D1.6mm_P2.54mm_Vertical, symbol Device:R
- added S?: EG1224 SPDT switch, SamacSys_Parts:EG1224, symbol SamacSys_Parts:EG1224
- added U?: D1213A-02SM, Package_TO_SOT_SMD:SOT-23-5_HandSoldering, symbol My_custom_lib:D1213A-02SM
Connections:
- net +3V3: now also R?.2, S?.2 (COM)
- net +BATT: now also BT?.1 (+), J?.1 (Pin_1), J?.1 (Pin_1), Q?.1 (S1)
- net +VDC: now also C?.1, D?.1 (K), IC?.8 (VIN), J?.3 (Pin_3), Q?.3 (S2), R?.2
- net GND: now also BT?.2 (-), C?.2, C?.2, D?.1 (K), D?.1 (K), D?.1 (K), IC?.6 (GND_1), IC?.7 (GND_2), J?.2 (Pin_2), J?.5 (GND), J?.6 (Shield), R?.1, S?.MH1, S?.MH2, S?.MH3, S?.MH4, U?.2 (VSS)
- new net: D?.2 (A), R?.1 (x3)
- new net: J?.2 (Pin_2), R?.2
- new net 3v3_enable: IC?.5 (EN), R?.1
- new net D+: J?.3 (D+), U?.4 (CH2)
- new net D-: J?.2 (D-), U?.3 (CH1)
- new net Drains: Q?.5 (D2_1), Q?.6 (D2_2), Q?.7 (D1_1), Q?.8 (D1_2)
- new net VBUS: D?.2 (A), FB?.2, Q?.2 (G1), Q?.4 (G2), R?.2, R?.2, U?.5 (VCC)
- new net VBUS_RAW: F?.1, J?.1 (VBUS)
- new net VBUS_RAW2: F?.2, FB?.1
- new net buck_out: S?.1 (PIN1)
- new net lin_reg: C?.1, IC?.1 (VOUT), S?.3 (PIN2)
- no-connect marks 3 -> 8
Other:
- added sheet buck (buck.kicad_sch)
- note added: "200-300mA <100 typical"
- note added: "400-500mA+ max power usage of MCU"
- note added: "BATT TO USB POWER AUTO SHITCHING WITH REVERSE POWER PROTECTION"
- note added: "ESD protection IC"
- note added: "Linear regulator just in case the buck fails or i need lower noise power"
- note added: "Power"
- note added: "Power indicator leds"
- note added: "USB Data+Power Input filtering and fuse"
- note added: "active high"

Commit message: j
Parts:
- removed BT?: Battery, symbol Device:Battery
- removed C17: 10u, symbol Device:C_Small
- removed C18, C19: 1u, Capacitor_SMD:C_0603_1608Metric_Pad1.08x0.95mm_HandSolder, symbol Device:C_Small
- removed C20: 47u, symbol Device:C_Small
- removed C23: 100n, Capacitor_SMD:C_0603_1608Metric_Pad1.08x0.95mm_HandSolder, symbol Device:C_Small
- removed D6: D_Shockley, Diode_THT:D_A-405_P12.70mm_Horizontal, symbol Device:D_Shockley
- removed IC3: AP2112M-3.3TRG1, SOIC127P600X170-8N, symbol SamacSys_Parts:AP2112M-3.3TRG1
- removed L1: 1uH, symbol pspice:INDUCTOR
- removed Q1, Q3: Q_PMOS_DGS, symbol Device:Q_PMOS_DGS
- removed R6: 10k, Resistor_SMD:R_0603_1608Metric_Pad0.98x0.95mm_HandSolder, symbol Device:R_Small
- removed R?: 4.7k, Resistor_THT:R_Axial_DIN0204_L3.6mm_D1.6mm_P2.54mm_Vertical, symbol Device:R
- removed SW1: RA12131100, symbol My_custom_lib:RA12131100
- removed SW2: SW_SPDT, symbol Switch:SW_SPDT
- added IC?: ISL9120IIAZ-TR5696, BGA9C40P3X3_141X141X55, symbol SamacSys_Parts:ISL9120IIAZ-TR5696
- added R? (x3): 10k, Resistor_SMD:R_0603_1608Metric_Pad0.98x0.95mm_HandSolder, symbol Device:R
- BT1: footprint Connector_PinHeader_2.54mm:PinHeader_1x02_P2.54mm_Vertical -> SamacSys_Parts:1043
- gave numbers to parts that had none: 19
Connections:
- net GND: now also R?.1
- net VBUS: now also R?.1, R?.2; no longer Q6.2 (G1)
- net at D17.2 (A): now also R?.1, R?.2
- new net: Q6.2 (G1), R?.2
- no-connect marks 8 -> 5
Other:
- note added: "Inverting charge pump"
- note added: "Li ion chargeing"
- note removed: "200-300mA <100 typical"
- note removed: "Maybe use the EN pins to swith power source?"
- note removed: "Will chose IC the day i order it + inductor"
- moved on the sheet: BT1, BT2, C21, C22, C34, C35, C36, C37, C5, C53, C54, C6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

Commit message: h
Parts:
- removed BT1: Battery_Cell, SamacSys_Parts:1043, symbol Device:Battery_Cell
- added U201: (no value), symbol My_custom_lib:APX810S05
- added U202: (no value), symbol SamacSys_Parts:1043
- RV201: renamed from RV1; value 4.7k -> (none); footprint Z_mycustom_footprint_lib:2002102255 -> (none)
- RV202: renamed from RV2; value 4.7k -> (none); footprint Z_mycustom_footprint_lib:2002102255 -> (none)
- gave numbers to parts that had none: 4
- renumbered BT2 to BT201, C21 to C201, C22 to C202, C53 to C203, C54 to C204, C5 to C205, C6 to C206, C34 to C207, C35 to C208, C36 to C209, C37 to C210, D2 to D201, D3 to D202, D4 to D203, D5 to D204, D16 to D205, D15 to D206, D17 to D207, D18 to D208, D10 to D209, D11 to D210, D19 to D211, F1 to F201, FB1 to FB201, FB3 to FB202, IC1 to IC201, IC2 to IC202, IC5 to IC204, J21 to J201, J13 to J202, J6 to J203, J7 to J204, J22 to J205, J23 to J206, Q6 to Q201, R7 to R201, R8 to R202, R9 to R203, R10 to R204, R76 to R206, R11 to R207, R12 to R208, R25 to R209, R26 to R210, R27 to R211, R28 to R212, R80 to R213, R78 to R216, R79 to R217, RTHT1 to RTHT201, RTHT2 to RTHT202, S6 to S201, U12 to U203, U7 to U204
Connections:
- net +BATT: now also U201.3 (Vcc), U202.1 (+)
- net GND: now also U201.2 (GND), U202.2 (-)
- net TE_ext: now reaches IC202.7 (~{PG(}TE))
- net TE_int: now reaches IC201.7 (~{PG(}TE))
- net at Q201.2 (G1), R205.2: now also U201.1 (RESET)
- no-connect marks 5 -> 8
Other:
- note removed: "Maybe use a higher V"
