File: RTC.kicad_sch (KiCad schematic)
At the start: 5 parts

Commit message: j
Parts:
- gave numbers to parts that had none: 5
Changed lines of the file:
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@@
   (symbol (lib_id "Device:Crystal_GND3_Small") (at 85.725 63.5 270) (unit 1)
     (in_bom yes) (on_board yes) (fields_autoplaced)
-    (property "Reference" "Y?" (id 0) (at 88.265 62.2299 90)
+    (property "Reference" "Y4" (id 0) (at 88.265 62.2299 90)
       (effects (font (size 1.27 1.27)) (justify left))
     )
@@
   (symbol (lib_id "Device:C") (at 74.93 60.96 90) (unit 1)
     (in_bom yes) (on_board yes)
-    (property "Reference" "C?" (id 0) (at 73.7616 58.039 0)
+    (property "Reference" "C59" (id 0) (at 73.7616 58.039 0)
       (effects (font (size 1.27 1.27)) (justify left))
     )
@@
   (symbol (lib_id "power:GND") (at 68.58 63.5 270) (unit 1)
     (in_bom yes) (on_board yes) (fields_autoplaced)
-    (property "Reference" "#PWR?" (id 0) (at 62.23 63.5 0)
+    (property "Reference" "#PWR0109" (id 0) (at 62.23 63.5 0)
       (effects (font (size 1.27 1.27)) hide)
     )
@@
   (symbol (lib_id "power:GND") (at 97.79 83.82 0) (unit 1)
     (in_bom yes) (on_board yes) (fields_autoplaced)
-    (property "Reference" "#PWR?" (id 0) (at 97.79 90.17 0)
+    (property "Reference" "#PWR0110" (id 0) (at 97.79 90.17 0)
       (effects (font (size 1.27 1.27)) hide)
     )
@@
   (symbol (lib_id "power:+3V3") (at 123.825 64.135 0) (unit 1)
     (in_bom yes) (on_board yes) (fields_autoplaced)
-    (property "Reference" "#PWR?" (id 0) (at 123.825 67.945 0)
+    (property "Reference" "#PWR0111" (id 0) (at 123.825 67.945 0)
       (effects (font (size 1.27 1.27)) hide)
     )
@@
   (symbol (lib_id "My_custom_lib:MCP79412") (at 113.03 66.675 0) (unit 1)
     (in_bom yes) (on_board yes) (fields_autoplaced)
-    (property "Reference" "U?" (id 0) (at 113.03 53.34 0))
+    (property "Reference" "U16" (id 0) (at 113.03 53.34 0))
     (property "Value" "MCP79412" (id 1) (at 113.03 55.88 0))
     (property "Footprint" "Package_SO:TSSOP-8_4.4x3mm_P0.65mm" (id 2) (at 114.3 55.245 0)
@@
   (symbol (lib_id "Device:Battery_Cell") (at 90.17 78.74 0) (unit 1)
     (in_bom yes) (on_board yes) (fields_autoplaced)
-    (property "Reference" "BT?" (id 0) (at 93.98 75.4379 0)
+    (property "Reference" "BT5" (id 0) (at 93.98 75.4379 0)
       (effects (font (size 1.27 1.27)) (justify left))
     )
@@
   (symbol (lib_id "Device:C") (at 74.93 67.31 90) (unit 1)
     (in_bom yes) (on_board yes)
-    (property "Reference" "C?" (id 0) (at 75.565 72.39 0)
+    (property "Reference" "C60" (id 0) (at 75.565 72.39 0)
       (effects (font (size 1.27 1.27)) (justify left))
     )

Commit message: h
Parts:
- renumbered BT5 to BT901, C59 to C901, C60 to C902, U16 to U901, Y4 to Y901
Changed lines of the file:
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@@
   (symbol (lib_id "Device:Crystal_GND3_Small") (at 85.725 63.5 270) (unit 1)
     (in_bom yes) (on_board yes) (fields_autoplaced)
-    (property "Reference" "Y4" (id 0) (at 88.265 62.2299 90)
+    (property "Reference" "Y901" (id 0) (at 88.265 62.2299 90)
       (effects (font (size 1.27 1.27)) (justify left))
     )
@@
   (symbol (lib_id "Device:C") (at 74.93 60.96 90) (unit 1)
     (in_bom yes) (on_board yes)
-    (property "Reference" "C59" (id 0) (at 73.7616 58.039 0)
+    (property "Reference" "C901" (id 0) (at 73.7616 58.039 0)
       (effects (font (size 1.27 1.27)) (justify left))
     )
@@
   (symbol (lib_id "power:GND") (at 68.58 63.5 270) (unit 1)
     (in_bom yes) (on_board yes) (fields_autoplaced)
-    (property "Reference" "#PWR0109" (id 0) (at 62.23 63.5 0)
+    (property "Reference" "#PWR0901" (id 0) (at 62.23 63.5 0)
       (effects (font (size 1.27 1.27)) hide)
     )
@@
   (symbol (lib_id "power:GND") (at 97.79 83.82 0) (unit 1)
     (in_bom yes) (on_board yes) (fields_autoplaced)
-    (property "Reference" "#PWR0110" (id 0) (at 97.79 90.17 0)
+    (property "Reference" "#PWR0902" (id 0) (at 97.79 90.17 0)
       (effects (font (size 1.27 1.27)) hide)
     )
@@
   (symbol (lib_id "power:+3V3") (at 123.825 64.135 0) (unit 1)
     (in_bom yes) (on_board yes) (fields_autoplaced)
-    (property "Reference" "#PWR0111" (id 0) (at 123.825 67.945 0)
+    (property "Reference" "#PWR0903" (id 0) (at 123.825 67.945 0)
       (effects (font (size 1.27 1.27)) hide)
     )
@@
   (symbol (lib_id "My_custom_lib:MCP79412") (at 113.03 66.675 0) (unit 1)
     (in_bom yes) (on_board yes) (fields_autoplaced)
-    (property "Reference" "U16" (id 0) (at 113.03 53.34 0))
+    (property "Reference" "U901" (id 0) (at 113.03 53.34 0))
     (property "Value" "MCP79412" (id 1) (at 113.03 55.88 0))
     (property "Footprint" "Package_SO:TSSOP-8_4.4x3mm_P0.65mm" (id 2) (at 114.3 55.245 0)
@@
   (symbol (lib_id "Device:Battery_Cell") (at 90.17 78.74 0) (unit 1)
     (in_bom yes) (on_board yes) (fields_autoplaced)
-    (property "Reference" "BT5" (id 0) (at 93.98 75.4379 0)
+    (property "Reference" "BT901" (id 0) (at 93.98 75.4379 0)
       (effects (font (size 1.27 1.27)) (justify left))
     )
@@
   (symbol (lib_id "Device:C") (at 74.93 67.31 90) (unit 1)
     (in_bom yes) (on_board yes)
-    (property "Reference" "C60" (id 0) (at 75.565 72.39 0)
+    (property "Reference" "C902" (id 0) (at 75.565 72.39 0)
       (effects (font (size 1.27 1.27)) (justify left))
     )
