File: buck.kicad_sch (KiCad schematic)
At the start: 8 parts

Commit message: j
Parts:
- gave numbers to parts that had none: 8
Changed lines of the file:
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@@
   (symbol (lib_id "Device:C_Small") (at 135.89 67.945 0) (unit 1)
     (in_bom yes) (on_board yes)
-    (property "Reference" "C?" (id 0) (at 129.54 66.675 0)
+    (property "Reference" "C56" (id 0) (at 129.54 66.675 0)
       (effects (font (size 1.27 1.27)) (justify left))
     )
@@
   (symbol (lib_id "power:GND") (at 66.04 72.39 0) (unit 1)
     (in_bom yes) (on_board yes) (fields_autoplaced)
-    (property "Reference" "#PWR?" (id 0) (at 66.04 78.74 0)
+    (property "Reference" "#PWR0104" (id 0) (at 66.04 78.74 0)
       (effects (font (size 1.27 1.27)) hide)
     )
@@
   (symbol (lib_id "power:GND") (at 86.36 74.93 0) (unit 1)
     (in_bom yes) (on_board yes) (fields_autoplaced)
-    (property "Reference" "#PWR?" (id 0) (at 86.36 81.28 0)
+    (property "Reference" "#PWR0105" (id 0) (at 86.36 81.28 0)
       (effects (font (size 1.27 1.27)) hide)
     )
@@
   (symbol (lib_id "Device:R_Small") (at 144.78 76.835 0) (unit 1)
     (in_bom yes) (on_board yes) (fields_autoplaced)
-    (property "Reference" "RR?" (id 0) (at 147.32 75.5649 0)
+    (property "Reference" "RR2" (id 0) (at 147.32 75.5649 0)
       (effects (font (size 1.27 1.27)) (justify left))
     )
@@
   (symbol (lib_id "My_custom_lib:DIO6012BCST6") (at 88.9 64.135 0) (unit 1)
     (in_bom yes) (on_board yes) (fields_autoplaced)
-    (property "Reference" "U?" (id 0) (at 88.9 53.34 0))
+    (property "Reference" "U15" (id 0) (at 88.9 53.34 0))
     (property "Value" "DIO6012BCST6" (id 1) (at 88.9 55.88 0))
     (property "Footprint" "Package_TO_SOT_SMD:SOT-23-6_Handsoldering" (id 2) (at 86.36 56.515 0)
@@
   (symbol (lib_id "Device:R_Small") (at 144.78 68.58 0) (unit 1)
     (in_bom yes) (on_board yes) (fields_autoplaced)
-    (property "Reference" "RR?" (id 0) (at 146.685 67.3099 0)
+    (property "Reference" "RR1" (id 0) (at 146.685 67.3099 0)
       (effects (font (size 1.27 1.27)) (justify left))
     )
@@
   (symbol (lib_id "Device:C_Small") (at 158.75 67.945 0) (unit 1)
     (in_bom yes) (on_board yes) (fields_autoplaced)
-    (property "Reference" "C?" (id 0) (at 161.29 66.6812 0)
+    (property "Reference" "C57" (id 0) (at 161.29 66.6812 0)
       (effects (font (size 1.27 1.27)) (justify left))
     )
@@
   (symbol (lib_id "Device:C_Small") (at 66.04 67.945 0) (unit 1)
     (in_bom yes) (on_board yes) (fields_autoplaced)
-    (property "Reference" "C?" (id 0) (at 68.58 66.6812 0)
+    (property "Reference" "C55" (id 0) (at 68.58 66.6812 0)
       (effects (font (size 1.27 1.27)) (justify left))
     )
@@
   (symbol (lib_id "power:GND") (at 144.78 81.28 0) (unit 1)
     (in_bom yes) (on_board yes) (fields_autoplaced)
-    (property "Reference" "#PWR?" (id 0) (at 144.78 87.63 0)
+    (property "Reference" "#PWR0106" (id 0) (at 144.78 87.63 0)
       (effects (font (size 1.27 1.27)) hide)
     )
@@
   (symbol (lib_id "Device:C_Small") (at 166.37 67.945 0) (unit 1)
     (in_bom yes) (on_board yes) (fields_autoplaced)
-    (property "Reference" "C?" (id 0) (at 168.91 66.6812 0)
+    (property "Reference" "C58" (id 0) (at 168.91 66.6812 0)
       (effects (font (size 1.27 1.27)) (justify left))
     )
@@
   (symbol (lib_id "power:GND") (at 158.75 73.025 0) (unit 1)
     (in_bom yes) (on_board yes) (fields_autoplaced)
-    (property "Reference" "#PWR?" (id 0) (at 158.75 79.375 0)
+    (property "Reference" "#PWR0107" (id 0) (at 158.75 79.375 0)
       (effects (font (size 1.27 1.27)) hide)
     )
@@
   (symbol (lib_id "SamacSys_Parts:NRH3012T2R2MN") (at 102.87 64.135 0) (unit 1)
     (in_bom yes) (on_board yes) (fields_autoplaced)
-    (property "Reference" "L?" (id 0) (at 113.03 57.785 0))
+    (property "Reference" "L2" (id 0) (at 113.03 57.785 0))
     (property "Value" "NRH3012T2R2MN  2,2uH" (id 1) (at 113.03 60.325 0))
     (property "Footprint" "SamacSys_Parts:NRH3012T220MNV" (id 2) (at 119.38 62.865 0)
@@
   (symbol (lib_id "power:GND") (at 166.37 73.025 0) (unit 1)
     (in_bom yes) (on_board yes) (fields_autoplaced)
-    (property "Reference" "#PWR?" (id 0) (at 166.37 79.375 0)
-      (effects (font (size 1.27 1.27)) hide)
-    )
+    (property "Reference" "#PWR0108" (id 0) (at 166.37 79.375 0)
+      (effects (font (size 1.27 1.27)) hide)
+    )

Commit message: h
Parts:
- renumbered C55 to C801, C56 to C802, C57 to C803, C58 to C804, L2 to L801, RR1 to RR801, RR2 to RR802, U15 to U801
Changed lines of the file:
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@@
   (symbol (lib_id "Device:C_Small") (at 135.89 67.945 0) (unit 1)
     (in_bom yes) (on_board yes)
-    (property "Reference" "C56" (id 0) (at 129.54 66.675 0)
+    (property "Reference" "C802" (id 0) (at 129.54 66.675 0)
       (effects (font (size 1.27 1.27)) (justify left))
     )
@@
   (symbol (lib_id "power:GND") (at 66.04 72.39 0) (unit 1)
     (in_bom yes) (on_board yes) (fields_autoplaced)
-    (property "Reference" "#PWR0104" (id 0) (at 66.04 78.74 0)
+    (property "Reference" "#PWR0801" (id 0) (at 66.04 78.74 0)
       (effects (font (size 1.27 1.27)) hide)
     )
@@
   (symbol (lib_id "power:GND") (at 86.36 74.93 0) (unit 1)
     (in_bom yes) (on_board yes) (fields_autoplaced)
-    (property "Reference" "#PWR0105" (id 0) (at 86.36 81.28 0)
+    (property "Reference" "#PWR0802" (id 0) (at 86.36 81.28 0)
       (effects (font (size 1.27 1.27)) hide)
     )
@@
   (symbol (lib_id "Device:R_Small") (at 144.78 76.835 0) (unit 1)
     (in_bom yes) (on_board yes) (fields_autoplaced)
-    (property "Reference" "RR2" (id 0) (at 147.32 75.5649 0)
+    (property "Reference" "RR802" (id 0) (at 147.32 75.5649 0)
       (effects (font (size 1.27 1.27)) (justify left))
     )
@@
   (symbol (lib_id "My_custom_lib:DIO6012BCST6") (at 88.9 64.135 0) (unit 1)
     (in_bom yes) (on_board yes) (fields_autoplaced)
-    (property "Reference" "U15" (id 0) (at 88.9 53.34 0))
+    (property "Reference" "U801" (id 0) (at 88.9 53.34 0))
     (property "Value" "DIO6012BCST6" (id 1) (at 88.9 55.88 0))
     (property "Footprint" "Package_TO_SOT_SMD:SOT-23-6_Handsoldering" (id 2) (at 86.36 56.515 0)
@@
   (symbol (lib_id "Device:R_Small") (at 144.78 68.58 0) (unit 1)
     (in_bom yes) (on_board yes) (fields_autoplaced)
-    (property "Reference" "RR1" (id 0) (at 146.685 67.3099 0)
+    (property "Reference" "RR801" (id 0) (at 146.685 67.3099 0)
       (effects (font (size 1.27 1.27)) (justify left))
     )
@@
   (symbol (lib_id "Device:C_Small") (at 158.75 67.945 0) (unit 1)
     (in_bom yes) (on_board yes) (fields_autoplaced)
-    (property "Reference" "C57" (id 0) (at 161.29 66.6812 0)
+    (property "Reference" "C803" (id 0) (at 161.29 66.6812 0)
       (effects (font (size 1.27 1.27)) (justify left))
     )
@@
   (symbol (lib_id "Device:C_Small") (at 66.04 67.945 0) (unit 1)
     (in_bom yes) (on_board yes) (fields_autoplaced)
-    (property "Reference" "C55" (id 0) (at 68.58 66.6812 0)
+    (property "Reference" "C801" (id 0) (at 68.58 66.6812 0)
       (effects (font (size 1.27 1.27)) (justify left))
     )
@@
   (symbol (lib_id "power:GND") (at 144.78 81.28 0) (unit 1)
     (in_bom yes) (on_board yes) (fields_autoplaced)
-    (property "Reference" "#PWR0106" (id 0) (at 144.78 87.63 0)
+    (property "Reference" "#PWR0803" (id 0) (at 144.78 87.63 0)
       (effects (font (size 1.27 1.27)) hide)
     )
@@
   (symbol (lib_id "Device:C_Small") (at 166.37 67.945 0) (unit 1)
     (in_bom yes) (on_board yes) (fields_autoplaced)
-    (property "Reference" "C58" (id 0) (at 168.91 66.6812 0)
+    (property "Reference" "C804" (id 0) (at 168.91 66.6812 0)
       (effects (font (size 1.27 1.27)) (justify left))
     )
@@
   (symbol (lib_id "power:GND") (at 158.75 73.025 0) (unit 1)
     (in_bom yes) (on_board yes) (fields_autoplaced)
-    (property "Reference" "#PWR0107" (id 0) (at 158.75 79.375 0)
+    (property "Reference" "#PWR0804" (id 0) (at 158.75 79.375 0)
       (effects (font (size 1.27 1.27)) hide)
     )
@@
   (symbol (lib_id "SamacSys_Parts:NRH3012T2R2MN") (at 102.87 64.135 0) (unit 1)
     (in_bom yes) (on_board yes) (fields_autoplaced)
-    (property "Reference" "L2" (id 0) (at 113.03 57.785 0))
+    (property "Reference" "L801" (id 0) (at 113.03 57.785 0))
     (property "Value" "NRH3012T2R2MN  2,2uH" (id 1) (at 113.03 60.325 0))
     (property "Footprint" "SamacSys_Parts:NRH3012T220MNV" (id 2) (at 119.38 62.865 0)
@@
   (symbol (lib_id "power:GND") (at 166.37 73.025 0) (unit 1)
     (in_bom yes) (on_board yes) (fields_autoplaced)
-    (property "Reference" "#PWR0108" (id 0) (at 166.37 79.375 0)
-      (effects (font (size 1.27 1.27)) hide)
-    )
+    (property "Reference" "#PWR0805" (id 0) (at 166.37 79.375 0)
+      (effects (font (size 1.27 1.27)) hide)
+    )
