File: multiplexing+gpio_extenders.kicad_sch (KiCad schematic)
At the start: 3 parts, among them IC4 PEC12R-4230F-S0024, U12 CD4052B, U13 CD4052B

Commit message: h
Parts:
- removed U12, U13: CD4052B, symbol Analog_Switch:CD4052B
- added IC?: XRA1203IG24TR-F, SOP65P640X120-24N, symbol SamacSys_Parts:XRA1203IG24TR-F
- added U? (x2): MC74VHC4052DR2G, Package_SO:SOIC-16_3.9x9.9mm_P1.27mm, symbol My_custom_lib:MC74VHC4052DR2G
Connections:
- no-connect marks 0 -> 2
Other:
- moved on the sheet: IC4

Commit message: j
Parts:
- gave numbers to parts that had none: 3
Changed lines of the file:
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@@
   (symbol (lib_id "SamacSys_Parts:XRA1203IG24TR-F") (at 73.025 131.445 0) (unit 1)
     (in_bom yes) (on_board yes) (fields_autoplaced)
-    (property "Reference" "IC?" (id 0) (at 88.265 123.19 0))
+    (property "Reference" "IC6" (id 0) (at 88.265 123.19 0))
     (property "Value" "XRA1203IG24TR-F" (id 1) (at 88.265 125.73 0))
     (property "Footprint" "SOP65P640X120-24N" (id 2) (at 99.695 128.905 0)
@@
   (symbol (lib_id "My_custom_lib:MC74VHC4052DR2G") (at 64.135 48.26 0) (unit 1)
     (in_bom yes) (on_board yes) (fields_autoplaced)
-    (property "Reference" "U?" (id 0) (at 63.5 29.845 0))
+    (property "Reference" "U13" (id 0) (at 63.5 29.845 0))
     (property "Value" "MC74VHC4052DR2G" (id 1) (at 63.5 32.385 0))
     (property "Footprint" "Package_SO:SOIC-16_3.9x9.9mm_P1.27mm" (id 2) (at 61.595 29.21 0)
@@
   (symbol (lib_id "My_custom_lib:MC74VHC4052DR2G") (at 158.115 50.165 0) (unit 1)
     (in_bom yes) (on_board yes) (fields_autoplaced)
-    (property "Reference" "U?" (id 0) (at 157.48 31.75 0))
+    (property "Reference" "U14" (id 0) (at 157.48 31.75 0))
     (property "Value" "MC74VHC4052DR2G" (id 1) (at 157.48 34.29 0))
     (property "Footprint" "Package_SO:SOIC-16_3.9x9.9mm_P1.27mm" (id 2) (at 155.575 31.115 0)

Commit message: h
Parts:
- added JP701: (no value), symbol Jumper:Jumper_2_Open
- added JP702: J1, Jumper:SolderJumper-2_P1.3mm_Open_RoundedPad1.0x1.5mm, symbol Jumper:Jumper_2_Open
- added R701, R702, R703, R704, R705: 10k, Resistor_SMD:R_0603_1608Metric_Pad0.98x0.95mm_HandSolder, symbol Device:R
- renumbered IC6 to IC701, IC4 to IC702, U13 to U701, U14 to U702
Connections:
- net ADC1: now also U701.13 (X_OUT)
- net ADC2: now also U701.3 (Y_OUT)
- net ADC3: now also U702.13 (X_OUT)
- net ADC4: now also U702.3 (Y_OUT)
- net COMP1: now also IC701.5 (P1)
- net COMP2: now also IC701.6 (P2)
- net COMP3: now also IC701.7 (P3)
- net COMP4: now also IC701.8 (P4)
- net COMP5: now also IC701.9 (P5)
- net COMP6: now also IC701.10 (P6)
- net LCD_CS: now also IC701.11 (P7)
- net LCD_RST: now also IC701.4 (P0)
- net bat1_v: now also U701.12 (X0)
- net bat2_v: now also U701.1 (Y0)
- net component1: now also U701.15 (X2)
- net component2: now also U701.2 (Y2)
- net component3: now also U702.15 (X2)
- net measured_batt_I: now also U702.1 (Y0)
- net measured_batt_v: now also U702.12 (X0)
- net mux1: now also IC701.13 (P8), U701.9 (B), U702.9 (B)
- net mux2: now also IC701.14 (P9), U701.10 (A), U702.10 (A)
- net scope1: now also U701.11 (X3)
- net scope2: now also U701.4 (Y3)
- net scope3: now also U702.11 (X3)
- net scope4: now also U702.4 (Y3)
- net thermistor: now also U702.2 (Y2)
- net IRQ: now reaches IC701.1 (IRQ#)
- net GND: now reaches IC701.12 (GND)
- net GND: now also U701.7 (VEE), U701.8 (GND), U702.7 (VEE), U702.8 (GND), JP701.1 (A), JP702.1 (A), R701.2, R702.2
- net enable1: now reaches IC701.15 (P10)
- net enable1: now also U701.6 (ENABLE), R701.1
- net enable2: now reaches IC701.16 (P11)
- net enable2: now also U702.6 (ENABLE), R702.1
- net A1: now reaches IC701.2 (A1)
- net A1: now also JP702.2 (B), R704.1
- net A0: now reaches IC701.21 (A0)
- net A0: now also JP701.2 (B), R703.1
- net SCL: now reaches IC701.22 (SCL)
- net SDA: now reaches IC701.23 (SDA)
- net +3V3: now reaches IC701.24 (VCC)
- net +3V3: now also U701.16 (VCC), U702.16 (VCC), R703.2, R704.2, R705.2
- net RESET: now reaches IC701.3 (RESET#)
- net RESET: now also R705.1
- no-connect marks 2 -> 6
Other:
- moved on the sheet: IC702
